File: clock.kicad_sch (KiCad schematic)
At the start: 24 parts

Commit message: Fix Clock
Parts:
- C1, C10, C3: value (none) -> 0.1µF; footprint (none) -> Capacitor_THT:C_Disc_D4.3mm_W1.9mm_P5.00mm
- C2, C4, C5: value (none) -> 0.01µF; footprint (none) -> Capacitor_THT:C_Disc_D4.3mm_W1.9mm_P5.00mm
- C6: value (none) -> 1µF; footprint (none) -> Capacitor_THT:CP_Radial_D5.0mm_P2.00mm; symbol Device:CP1 -> Device:C
- D1: value (none) -> BLUE; footprint (none) -> LED_THT:LED_D5.0mm; symbol Device:LED_ALT -> Device:LED
- R1, R2, R3, R5, R6: value (none) -> 1K; footprint (none) -> Resistor_THT:R_Axial_DIN0207_L6.3mm_D2.5mm_P7.62mm_Horizontal
- R4: value (none) -> 1M; footprint (none) -> Resistor_THT:R_Axial_DIN0207_L6.3mm_D2.5mm_P7.62mm_Horizontal
- R7: value (none) -> 220; footprint (none) -> Resistor_THT:R_Axial_DIN0207_L6.3mm_D2.5mm_P7.62mm_Horizontal
- RV1: value (none) -> 1M; footprint (none) -> 8bit-custom-footprints:Potentiometer-5.5mm; symbol 8bit-computer-rescue:POT -> Device:R_Potentiometer
- SW1: value (none) -> SW_Push; footprint (none) -> Button_Switch_THT:SW_PUSH_6mm_H5mm; symbol 8bit-computer-rescue:SW_Push -> Switch:SW_Push
- SW2: value (none) -> SW_SPDT; footprint (none) -> 8bit-custom-footprints:DPDT-pushbutton; symbol 8bit-computer-rescue:SW_SPDT -> Switch:SW_SPDT
- U1, U2, U3: value (none) -> LM555; footprint (none) -> Package_DIP:DIP-8_W7.62mm; symbol 8bit-computer-rescue:LM555 -> Timer:LM555xN
- U4: value (none) -> 74LS04; footprint (none) -> Package_DIP:DIP-14_W7.62mm; symbol 8bit-computer-rescue:74LS04 -> 74xx:74LS04
- U5: value (none) -> 74LS08; footprint (none) -> Package_DIP:DIP-14_W7.62mm; symbol 8bit-computer-rescue:74LS08 -> 74xx:74LS08
- U6: value (none) -> 74LS32; footprint (none) -> Package_DIP:DIP-14_W7.62mm; symbol 8bit-computer-rescue:74LS32 -> 74xx:74LS32
Connections:
- net CLK: now also D1.2 (A), U4.3, U5.8
- net GND: now also C6.2, SW1.1, SW2.2 (B), U1.1 (GND), U2.1 (GND), U3.1 (GND), U3.6 (THR)
- net HLT: now also U4.5
- net VCC: now also U1.4 (R), U1.8 (VCC), U2.4 (R), U2.8 (VCC), U3.8 (VCC)
- net ~{CLK}: now also U4.4
- net at R1.2, R2.2: now also U1.7 (DIS)
- net at R3.2: now also SW1.2, U2.2 (TR)
- net at R6.2: now also SW2.3 (C), U3.4 (R)
- net at R5.2: now also SW2.1 (A), U3.2 (TR)
- net at C3.1, R4.2: now also U2.6 (THR), U2.7 (DIS)
- net at C5.1: now also U1.5 (CV)
- net at C2.1: now also U2.5 (CV)
- net at C4.1: now also U3.5 (CV)
- net at R7.1: now also D1.1 (K)
- net at R2.1: now also RV1.2
- new net: C6.1, RV1.1, U1.2 (TR), U1.6 (THR)
- new net: U1.3 (Q), U5.1
- new net: U3.3 (Q), U4.1, U5.2
- new net: U2.3 (Q), U5.5
- new net: U4.2, U5.4
- new net: U5.3, U6.1
- new net: U5.6, U6.2
- new net: U5.9, U6.3
- new net: U4.6, U5.10
- no-connect marks 20 -> 2
Other:
- title: (none) -> Clock
