File: a-register.kicad_sch (KiCad schematic)
At the start: 20 parts

Commit message: Fix Clock
Parts:
- C11: value (none) -> 0.1µF; footprint (none) -> Capacitor_THT:C_Disc_D4.3mm_W1.9mm_P5.00mm
- D10, D11, D12, D13, D14, D15, D16, D17: value (none) -> RED; footprint (none) -> LED_THT:LED_D5.0mm
- R24, R25, R26, R27, R28, R29, R30, R31: value (none) -> 220; footprint (none) -> Resistor_THT:R_Axial_DIN0207_L6.3mm_D2.5mm_P7.62mm_Horizontal
- U7: value (none) -> 74LS245; footprint (none) -> Package_DIP:DIP-20_W7.62mm
- U8, U9: value (none) -> 74LS173; footprint (none) -> Package_DIP:DIP-16_W7.62mm
Changed lines of the file:
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@@
     (in_bom yes) (on_board yes)
     (property "Reference" "U8" (id 0) (at 135.89 71.12 0))
-    (property "Value" "" (id 1) (at 132.08 71.12 0))
-    (property "Footprint" "" (id 2) (at 133.35 68.58 0)
+    (property "Value" "74LS173" (id 1) (at 132.08 71.12 0))
+    (property "Footprint" "Package_DIP:DIP-16_W7.62mm" (id 2) (at 133.35 68.58 0)
       (effects (font (size 1.27 1.27)) hide)
     )
@@
     (in_bom yes) (on_board yes)
     (property "Reference" "D12" (id 0) (at 111.76 142.24 0))
-    (property "Value" "" (id 1) (at 116.84 142.24 0))
-    (property "Footprint" "" (id 2) (at 114.3 142.24 0)
+    (property "Value" "RED" (id 1) (at 116.84 142.24 0))
+    (property "Footprint" "LED_THT:LED_D5.0mm" (id 2) (at 114.3 142.24 0)
       (effects (font (size 1.27 1.27)) hide)
     )
@@
     (in_bom yes) (on_board yes)
     (property "Reference" "D16" (id 0) (at 142.24 142.24 0))
-    (property "Value" "" (id 1) (at 147.32 142.24 0))
-    (property "Footprint" "" (id 2) (at 144.78 142.24 0)
+    (property "Value" "RED" (id 1) (at 147.32 142.24 0))
+    (property "Footprint" "LED_THT:LED_D5.0mm" (id 2) (at 144.78 142.24 0)
       (effects (font (size 1.27 1.27)) hide)
     )
@@
     (in_bom yes) (on_board yes)
     (property "Reference" "D17" (id 0) (at 149.86 142.24 0))
-    (property "Value" "" (id 1) (at 154.94 142.24 0))
-    (property "Footprint" "" (id 2) (at 152.4 142.24 0)
+    (property "Value" "RED" (id 1) (at 154.94 142.24 0))
+    (property "Footprint" "LED_THT:LED_D5.0mm" (id 2) (at 152.4 142.24 0)
       (effects (font (size 1.27 1.27)) hide)
     )
@@
     (in_bom yes) (on_board yes)
     (property "Reference" "R26" (id 0) (at 116.332 153.67 90))
-    (property "Value" "" (id 1) (at 114.3 153.67 90))
-    (property "Footprint" "" (id 2) (at 112.522 153.67 90)
+    (property "Value" "220" (id 1) (at 114.3 153.67 90))
+    (property "Footprint" "Resistor_THT:R_Axial_DIN0207_L6.3mm_D2.5mm_P7.62mm_Horizontal" (id 2) (at 112.522 153.67 90)
       (effects (font (size 1.27 1.27)) hide)
     )
@@
     (in_bom yes) (on_board yes)
     (property "Reference" "R27" (id 0) (at 123.952 153.67 90))
-    (property "Value" "" (id 1) (at 121.92 153.67 90))
-    (property "Footprint" "" (id 2) (at 120.142 153.67 90)
+    (property "Value" "220" (id 1) (at 121.92 153.67 90))
+    (property "Footprint" "Resistor_THT:R_Axial_DIN0207_L6.3mm_D2.5mm_P7.62mm_Horizontal" (id 2) (at 120.142 153.67 90)
       (effects (font (size 1.27 1.27)) hide)
     )
@@
     (in_bom yes) (on_board yes)
     (property "Reference" "R29" (id 0) (at 139.192 153.67 90))
-    (property "Value" "" (id 1) (at 137.16 153.67 90))
-    (property "Footprint" "" (id 2) (at 135.382 153.67 90)
+    (property "Value" "220" (id 1) (at 137.16 153.67 90))
+    (property "Footprint" "Resistor_THT:R_Axial_DIN0207_L6.3mm_D2.5mm_P7.62mm_Horizontal" (id 2) (at 135.382 153.67 90)
       (effects (font (size 1.27 1.27)) hide)
     )
@@
     (in_bom yes) (on_board yes)
     (property "Reference" "R31" (id 0) (at 154.432 153.67 90))
-    (property "Value" "" (id 1) (at 152.4 153.67 90))
-    (property "Footprint" "" (id 2) (at 150.622 153.67 90)
+    (property "Value" "220" (id 1) (at 152.4 153.67 90))
+    (property "Footprint" "Resistor_THT:R_Axial_DIN0207_L6.3mm_D2.5mm_P7.62mm_Horizontal" (id 2) (at 150.622 153.67 90)
       (effects (font (size 1.27 1.27)) hide)
     )
@@
       (effects (font (size 1.27 1.27)) hide)
     )
-    (property "Value" "" (id 1) (at 109.22 73.66 0))
+    (property "Value" "VCC" (id 1) (at 109.22 73.66 0))
     (property "Footprint" "" (id 2) (at 109.22 77.47 0)
       (effects (font (size 1.27 1.27)) hide)
@@
     (in_bom yes) (on_board yes)
     (property "Reference" "U9" (id 0) (at 176.53 71.12 0))
-    (property "Value" "" (id 1) (at 172.72 71.12 0))
-    (property "Footprint" "" (id 2) (at 173.99 68.58 0)
+    (property "Value" "74LS173" (id 1) (at 172.72 71.12 0))
+    (property "Footprint" "Package_DIP:DIP-16_W7.62mm" (id 2) (at 173.99 68.58 0)
       (effects (font (size 1.27 1.27)) hide)
     )
@@
       (effects (font (size 1.27 1.27)) (justify left bottom))
     )
-    (property "Value" "" (id 1) (at 106.045 67.31 0)
+    (property "Value" "74LS245" (id 1) (at 106.045 67.31 0)
       (effects (font (size 1.27 1.27)) (justify left top))
     )
-    (property "Footprint" "" (id 2) (at 91.44 68.58 0)
+    (property "Footprint" "Package_DIP:DIP-20_W7.62mm" (id 2) (at 91.44 68.58 0)
       (effects (font (size 1.27 1.27)) hide)
     )
@@
     (in_bom yes) (on_board yes)
     (property "Reference" "D10" (id 0) (at 96.52 142.24 0))
-    (property "Value" "" (id 1) (at 101.6 142.24 0))
-    (property "Footprint" "" (id 2) (at 99.06 142.24 0)
+    (property "Value" "RED" (id 1) (at 101.6 142.24 0))
+    (property "Footprint" "LED_THT:LED_D5.0mm" (id 2) (at 99.06 142.24 0)
       (effects (font (size 1.27 1.27)) hide)
     )
@@
     (in_bom yes) (on_board yes)
     (property "Reference" "D11" (id 0) (at 104.14 142.24 0))
-    (property "Value" "" (id 1) (at 109.22 142.24 0))
-    (property "Footprint" "" (id 2) (at 106.68 142.24 0)
+    (property "Value" "RED" (id 1) (at 109.22 142.24 0))
+    (property "Footprint" "LED_THT:LED_D5.0mm" (id 2) (at 106.68 142.24 0)
       (effects (font (size 1.27 1.27)) hide)
     )
@@
     (in_bom yes) (on_board yes)
     (property "Reference" "D13" (id 0) (at 119.38 142.24 0))
-    (property "Value" "" (id 1) (at 124.46 142.24 0))
-    (property "Footprint" "" (id 2) (at 121.92 142.24 0)
+    (property "Value" "RED" (id 1) (at 124.46 142.24 0))
+    (property "Footprint" "LED_THT:LED_D5.0mm" (id 2) (at 121.92 142.24 0)
       (effects (font (size 1.27 1.27)) hide)
     )
@@
     (in_bom yes) (on_board yes)
     (property "Reference" "D14" (id 0) (at 127 142.24 0))
-    (property "Value" "" (id 1) (at 132.08 142.24 0))
-    (property "Footprint" "" (id 2) (at 129.54 142.24 0)
+    (property "Value" "RED" (id 1) (at 132.08 142.24 0))
+    (property "Footprint" "LED_THT:LED_D5.0mm" (id 2) (at 129.54 142.24 0)
       (effects (font (size 1.27 1.27)) hide)
     )
@@
     (in_bom yes) (on_board yes)
     (property "Reference" "D15" (id 0) (at 134.62 142.24 0))
-    (property "Value" "" (id 1) (at 139.7 142.24 0))
-    (property "Footprint" "" (id 2) (at 137.16 142.24 0)
+    (property "Value" "RED" (id 1) (at 139.7 142.24 0))
+    (property "Footprint" "LED_THT:LED_D5.0mm" (id 2) (at 137.16 142.24 0)
       (effects (font (size 1.27 1.27)) hide)
     )
@@
     (in_bom yes) (on_board yes)
     (property "Reference" "R24" (id 0) (at 101.092 153.67 90))
-    (property "Value" "" (id 1) (at 99.06 153.67 90))
-    (property "Footprint" "" (id 2) (at 97.282 153.67 90)
+    (property "Value" "220" (id 1) (at 99.06 153.67 90))
+    (property "Footprint" "Resistor_THT:R_Axial_DIN0207_L6.3mm_D2.5mm_P7.62mm_Horizontal" (id 2) (at 97.282 153.67 90)
       (effects (font (size 1.27 1.27)) hide)
     )
@@
     (in_bom yes) (on_board yes)
     (property "Reference" "R25" (id 0) (at 108.712 153.67 90))
-    (property "Value" "" (id 1) (at 106.68 153.67 90))
-    (property "Footprint" "" (id 2) (at 104.902 153.67 90)
+    (property "Value" "220" (id 1) (at 106.68 153.67 90))
+    (property "Footprint" "Resistor_THT:R_Axial_DIN0207_L6.3mm_D2.5mm_P7.62mm_Horizontal" (id 2) (at 104.902 153.67 90)
       (effects (font (size 1.27 1.27)) hide)
     )
@@
     (in_bom yes) (on_board yes)
     (property "Reference" "R28" (id 0) (at 131.572 153.67 90))
-    (property "Value" "" (id 1) (at 129.54 153.67 90))
-    (property "Footprint" "" (id 2) (at 127.762 153.67 90)
+    (property "Value" "220" (id 1) (at 129.54 153.67 90))
+    (property "Footprint" "Resistor_THT:R_Axial_DIN0207_L6.3mm_D2.5mm_P7.62mm_Horizontal" (id 2) (at 127.762 153.67 90)
       (effects (font (size 1.27 1.27)) hide)
     )
@@
     (in_bom yes) (on_board yes)
     (property "Reference" "R30" (id 0) (at 146.812 153.67 90))
-    (property "Value" "" (id 1) (at 144.78 153.67 90))
-    (property "Footprint" "" (id 2) (at 143.002 153.67 90)
+    (property "Value" "220" (id 1) (at 144.78 153.67 90))
+    (property "Footprint" "Resistor_THT:R_Axial_DIN0207_L6.3mm_D2.5mm_P7.62mm_Horizontal" (id 2) (at 143.002 153.67 90)
       (effects (font (size 1.27 1.27)) hide)
     )
@@
       (effects (font (size 1.27 1.27)) hide)
     )
-    (property "Value" "" (id 1) (at 125.73 170.18 0))
+    (property "Value" "GND" (id 1) (at 125.73 170.18 0))
     (property "Footprint" "" (id 2) (at 125.73 166.37 0)
       (effects (font (size 1.27 1.27)) hide)
@@
       (effects (font (size 1.27 1.27)) hide)
     )
-    (property "Value" "" (id 1) (at 195.58 59.69 0))
+    (property "Value" "GND" (id 1) (at 195.58 59.69 0))
     (property "Footprint" "" (id 2) (at 195.58 55.88 0)
       (effects (font (size 1.27 1.27)) hide)
@@
       (effects (font (size 1.27 1.27)) (justify left))
     )
-    (property "Value" "" (id 1) (at 231.775 69.85 0)
+    (property "Value" "0.1µF" (id 1) (at 231.775 69.85 0)
       (effects (font (size 1.27 1.27)) (justify left))
     )
-    (property "Footprint" "" (id 2) (at 232.1052 71.12 0)
+    (property "Footprint" "Capacitor_THT:C_Disc_D4.3mm_W1.9mm_P5.00mm" (id 2) (at 232.1052 71.12 0)
       (effects (font (size 1.27 1.27)) hide)
     )
@@
       (effects (font (size 1.27 1.27)) hide)
     )
-    (property "Value" "" (id 1) (at 231.14 77.47 0))
+    (property "Value" "GND" (id 1) (at 231.14 77.47 0))
     (property "Footprint" "" (id 2) (at 231.14 73.66 0)
       (effects (font (size 1.27 1.27)) hide)
@@
       (effects (font (size 1.27 1.27)) hide)
     )
-    (property "Value" "" (id 1) (at 231.14 57.15 0))
+    (property "Value" "VCC" (id 1) (at 231.14 57.15 0))
     (property "Footprint" "" (id 2) (at 231.14 60.96 0)
       (effects (font (size 1.27 1.27)) hide)

Commit message: Fix
Parts:
- D10, D11, D12, D13, D14, D15, D16, D17: symbol Device:LED_ALT -> Device:LED
- U7: symbol 8bit-computer-rescue:74LS245 -> 74xx:74LS245
- U8, U9: symbol 8bit-computer-rescue:74LS173 -> 74xx:74LS173
Connections:
- net A_0: now also D17.2 (A), U7.9 (A7), U9.6 (Q3)
- net A_1: now also D16.2 (A), U7.8 (A6), U9.5 (Q2)
- net A_2: now also D15.2 (A), U7.7 (A5), U9.4 (Q1)
- net A_3: now also D14.2 (A), U7.6 (A4), U9.3 (Q0)
- net A_4: now also D13.2 (A), U7.5 (A3), U8.6 (Q3)
- net A_5: now also D12.2 (A), U7.4 (A2), U8.5 (Q2)
- net A_6: now also D11.2 (A), U7.3 (A1), U8.4 (Q1)
- net A_7: now also D10.2 (A), U7.2 (A0), U8.3 (Q0)
- net BUS_0: now also U7.11 (B7), U9.11 (D3)
- net BUS_1: now also U7.12 (B6), U9.12 (D2)
- net BUS_2: now also U7.13 (B5), U9.13 (D1)
- net BUS_3: now also U7.14 (B4), U9.14 (D0)
- net BUS_4: now also U7.15 (B3), U8.11 (D3)
- net BUS_5: now also U7.16 (B2), U8.12 (D2)
- net BUS_6: now also U7.17 (B1), U8.13 (D1)
- net BUS_7: now also U7.18 (B0), U8.14 (D0)
- net CLK: now also U8.7 (Cp), U9.7 (Cp)
- net CLR: now also U8.15 (Mr), U9.15 (Mr)
- net GND: now also U8.1 (Oe1), U8.2 (Oe2), U9.1 (Oe1), U9.2 (Oe2)
- net VCC: now also U7.1 (A->B)
- net ~{AI}: now also U8.10 (E2), U8.9 (E1), U9.10 (E2), U9.9 (E1)
- net ~{AO}: now also U7.19 (CE)
- net at R26.1: now also D12.1 (K)
- net at R27.1: now also D13.1 (K)
- net at R29.1: now also D15.1 (K)
- net at R31.1: now also D17.1 (K)
- net at R24.1: now also D10.1 (K)
- net at R25.1: now also D11.1 (K)
- net at R28.1: now also D14.1 (K)
- net at R30.1: now also D16.1 (K)
