File: b-register.kicad_sch (KiCad schematic)
At the start: 20 parts

Commit message: Fix Clock
Parts:
- C12: value (none) -> 0.1µF; footprint (none) -> Capacitor_THT:C_Disc_D4.3mm_W1.9mm_P5.00mm
- D18, D19, D20, D21, D22, D23, D24, D25: value (none) -> RED; footprint (none) -> LED_THT:LED_D5.0mm
- R32, R33, R34, R35, R36, R37, R38, R39: value (none) -> 220; footprint (none) -> Resistor_THT:R_Axial_DIN0207_L6.3mm_D2.5mm_P7.62mm_Horizontal
- U10: value (none) -> 74LS245; footprint (none) -> Package_DIP:DIP-20_W7.62mm
- U11, U12: value (none) -> 74LS173; footprint (none) -> Package_DIP:DIP-16_W7.62mm
Changed lines of the file:
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@@
     (in_bom yes) (on_board yes)
     (property "Reference" "U12" (id 0) (at 176.53 68.58 0))
-    (property "Value" "" (id 1) (at 172.72 68.58 0))
-    (property "Footprint" "" (id 2) (at 173.99 66.04 0)
+    (property "Value" "74LS173" (id 1) (at 172.72 68.58 0))
+    (property "Footprint" "Package_DIP:DIP-16_W7.62mm" (id 2) (at 173.99 66.04 0)
       (effects (font (size 1.27 1.27)) hide)
     )
@@
       (effects (font (size 1.27 1.27)) (justify left bottom))
     )
-    (property "Value" "" (id 1) (at 106.045 64.77 0)
+    (property "Value" "74LS245" (id 1) (at 106.045 64.77 0)
       (effects (font (size 1.27 1.27)) (justify left top))
     )
-    (property "Footprint" "" (id 2) (at 91.44 66.04 0)
+    (property "Footprint" "Package_DIP:DIP-20_W7.62mm" (id 2) (at 91.44 66.04 0)
       (effects (font (size 1.27 1.27)) hide)
     )
@@
     (in_bom yes) (on_board yes)
     (property "Reference" "D19" (id 0) (at 104.14 139.7 0))
-    (property "Value" "" (id 1) (at 109.22 139.7 0))
-    (property "Footprint" "" (id 2) (at 106.68 139.7 0)
+    (property "Value" "RED" (id 1) (at 109.22 139.7 0))
+    (property "Footprint" "LED_THT:LED_D5.0mm" (id 2) (at 106.68 139.7 0)
       (effects (font (size 1.27 1.27)) hide)
     )
@@
     (in_bom yes) (on_board yes)
     (property "Reference" "R32" (id 0) (at 101.092 151.13 90))
-    (property "Value" "" (id 1) (at 99.06 151.13 90))
-    (property "Footprint" "" (id 2) (at 97.282 151.13 90)
+    (property "Value" "220" (id 1) (at 99.06 151.13 90))
+    (property "Footprint" "Resistor_THT:R_Axial_DIN0207_L6.3mm_D2.5mm_P7.62mm_Horizontal" (id 2) (at 97.282 151.13 90)
       (effects (font (size 1.27 1.27)) hide)
     )
@@
     (in_bom yes) (on_board yes)
     (property "Reference" "R33" (id 0) (at 108.712 151.13 90))
-    (property "Value" "" (id 1) (at 106.68 151.13 90))
-    (property "Footprint" "" (id 2) (at 104.902 151.13 90)
+    (property "Value" "220" (id 1) (at 106.68 151.13 90))
+    (property "Footprint" "Resistor_THT:R_Axial_DIN0207_L6.3mm_D2.5mm_P7.62mm_Horizontal" (id 2) (at 104.902 151.13 90)
       (effects (font (size 1.27 1.27)) hide)
     )
@@
     (in_bom yes) (on_board yes)
     (property "Reference" "R38" (id 0) (at 146.812 151.13 90))
-    (property "Value" "" (id 1) (at 144.78 151.13 90))
-    (property "Footprint" "" (id 2) (at 143.002 151.13 90)
+    (property "Value" "220" (id 1) (at 144.78 151.13 90))
+    (property "Footprint" "Resistor_THT:R_Axial_DIN0207_L6.3mm_D2.5mm_P7.62mm_Horizontal" (id 2) (at 143.002 151.13 90)
       (effects (font (size 1.27 1.27)) hide)
     )
@@
       (effects (font (size 1.27 1.27)) hide)
     )
-    (property "Value" "" (id 1) (at 125.73 167.64 0))
+    (property "Value" "GND" (id 1) (at 125.73 167.64 0))
     (property "Footprint" "" (id 2) (at 125.73 163.83 0)
       (effects (font (size 1.27 1.27)) hide)
@@
       (effects (font (size 1.27 1.27)) hide)
     )
-    (property "Value" "" (id 1) (at 195.58 57.15 0))
+    (property "Value" "GND" (id 1) (at 195.58 57.15 0))
     (property "Footprint" "" (id 2) (at 195.58 53.34 0)
       (effects (font (size 1.27 1.27)) hide)
@@
     (in_bom yes) (on_board yes)
     (property "Reference" "U11" (id 0) (at 135.89 68.58 0))
-    (property "Value" "" (id 1) (at 132.08 68.58 0))
-    (property "Footprint" "" (id 2) (at 133.35 66.04 0)
+    (property "Value" "74LS173" (id 1) (at 132.08 68.58 0))
+    (property "Footprint" "Package_DIP:DIP-16_W7.62mm" (id 2) (at 133.35 66.04 0)
       (effects (font (size 1.27 1.27)) hide)
     )
@@
     (in_bom yes) (on_board yes)
     (property "Reference" "D18" (id 0) (at 96.52 139.7 0))
-    (property "Value" "" (id 1) (at 101.6 139.7 0))
-    (property "Footprint" "" (id 2) (at 99.06 139.7 0)
+    (property "Value" "RED" (id 1) (at 101.6 139.7 0))
+    (property "Footprint" "LED_THT:LED_D5.0mm" (id 2) (at 99.06 139.7 0)
       (effects (font (size 1.27 1.27)) hide)
     )
@@
     (in_bom yes) (on_board yes)
     (property "Reference" "D20" (id 0) (at 111.76 139.7 0))
-    (property "Value" "" (id 1) (at 116.84 139.7 0))
-    (property "Footprint" "" (id 2) (at 114.3 139.7 0)
+    (property "Value" "RED" (id 1) (at 116.84 139.7 0))
+    (property "Footprint" "LED_THT:LED_D5.0mm" (id 2) (at 114.3 139.7 0)
       (effects (font (size 1.27 1.27)) hide)
     )
@@
     (in_bom yes) (on_board yes)
     (property "Reference" "D21" (id 0) (at 119.38 139.7 0))
-    (property "Value" "" (id 1) (at 124.46 139.7 0))
-    (property "Footprint" "" (id 2) (at 121.92 139.7 0)
+    (property "Value" "RED" (id 1) (at 124.46 139.7 0))
+    (property "Footprint" "LED_THT:LED_D5.0mm" (id 2) (at 121.92 139.7 0)
       (effects (font (size 1.27 1.27)) hide)
     )
@@
     (in_bom yes) (on_board yes)
     (property "Reference" "D22" (id 0) (at 127 139.7 0))
-    (property "Value" "" (id 1) (at 132.08 139.7 0))
-    (property "Footprint" "" (id 2) (at 129.54 139.7 0)
+    (property "Value" "RED" (id 1) (at 132.08 139.7 0))
+    (property "Footprint" "LED_THT:LED_D5.0mm" (id 2) (at 129.54 139.7 0)
       (effects (font (size 1.27 1.27)) hide)
     )
@@
     (in_bom yes) (on_board yes)
     (property "Reference" "D23" (id 0) (at 134.62 139.7 0))
-    (property "Value" "" (id 1) (at 139.7 139.7 0))
-    (property "Footprint" "" (id 2) (at 137.16 139.7 0)
+    (property "Value" "RED" (id 1) (at 139.7 139.7 0))
+    (property "Footprint" "LED_THT:LED_D5.0mm" (id 2) (at 137.16 139.7 0)
       (effects (font (size 1.27 1.27)) hide)
     )
@@
     (in_bom yes) (on_board yes)
     (property "Reference" "D24" (id 0) (at 142.24 139.7 0))
-    (property "Value" "" (id 1) (at 147.32 139.7 0))
-    (property "Footprint" "" (id 2) (at 144.78 139.7 0)
+    (property "Value" "RED" (id 1) (at 147.32 139.7 0))
+    (property "Footprint" "LED_THT:LED_D5.0mm" (id 2) (at 144.78 139.7 0)
       (effects (font (size 1.27 1.27)) hide)
     )
@@
     (in_bom yes) (on_board yes)
     (property "Reference" "D25" (id 0) (at 149.86 139.7 0))
-    (property "Value" "" (id 1) (at 154.94 139.7 0))
-    (property "Footprint" "" (id 2) (at 152.4 139.7 0)
+    (property "Value" "RED" (id 1) (at 154.94 139.7 0))
+    (property "Footprint" "LED_THT:LED_D5.0mm" (id 2) (at 152.4 139.7 0)
       (effects (font (size 1.27 1.27)) hide)
     )
@@
     (in_bom yes) (on_board yes)
     (property "Reference" "R34" (id 0) (at 116.332 151.13 90))
-    (property "Value" "" (id 1) (at 114.3 151.13 90))
-    (property "Footprint" "" (id 2) (at 112.522 151.13 90)
+    (property "Value" "220" (id 1) (at 114.3 151.13 90))
+    (property "Footprint" "Resistor_THT:R_Axial_DIN0207_L6.3mm_D2.5mm_P7.62mm_Horizontal" (id 2) (at 112.522 151.13 90)
       (effects (font (size 1.27 1.27)) hide)
     )
@@
     (in_bom yes) (on_board yes)
     (property "Reference" "R35" (id 0) (at 123.952 151.13 90))
-    (property "Value" "" (id 1) (at 121.92 151.13 90))
-    (property "Footprint" "" (id 2) (at 120.142 151.13 90)
+    (property "Value" "220" (id 1) (at 121.92 151.13 90))
+    (property "Footprint" "Resistor_THT:R_Axial_DIN0207_L6.3mm_D2.5mm_P7.62mm_Horizontal" (id 2) (at 120.142 151.13 90)
       (effects (font (size 1.27 1.27)) hide)
     )
@@
     (in_bom yes) (on_board yes)
     (property "Reference" "R36" (id 0) (at 131.572 151.13 90))
-    (property "Value" "" (id 1) (at 129.54 151.13 90))
-    (property "Footprint" "" (id 2) (at 127.762 151.13 90)
+    (property "Value" "220" (id 1) (at 129.54 151.13 90))
+    (property "Footprint" "Resistor_THT:R_Axial_DIN0207_L6.3mm_D2.5mm_P7.62mm_Horizontal" (id 2) (at 127.762 151.13 90)
       (effects (font (size 1.27 1.27)) hide)
     )
@@
     (in_bom yes) (on_board yes)
     (property "Reference" "R37" (id 0) (at 139.192 151.13 90))
-    (property "Value" "" (id 1) (at 137.16 151.13 90))
-    (property "Footprint" "" (id 2) (at 135.382 151.13 90)
+    (property "Value" "220" (id 1) (at 137.16 151.13 90))
+    (property "Footprint" "Resistor_THT:R_Axial_DIN0207_L6.3mm_D2.5mm_P7.62mm_Horizontal" (id 2) (at 135.382 151.13 90)
       (effects (font (size 1.27 1.27)) hide)
     )
@@
     (in_bom yes) (on_board yes)
     (property "Reference" "R39" (id 0) (at 154.432 151.13 90))
-    (property "Value" "" (id 1) (at 152.4 151.13 90))
-    (property "Footprint" "" (id 2) (at 150.622 151.13 90)
+    (property "Value" "220" (id 1) (at 152.4 151.13 90))
+    (property "Footprint" "Resistor_THT:R_Axial_DIN0207_L6.3mm_D2.5mm_P7.62mm_Horizontal" (id 2) (at 150.622 151.13 90)
       (effects (font (size 1.27 1.27)) hide)
     )
@@
       (effects (font (size 1.27 1.27)) hide)
     )
-    (property "Value" "" (id 1) (at 109.22 71.12 0))
+    (property "Value" "VCC" (id 1) (at 109.22 71.12 0))
     (property "Footprint" "" (id 2) (at 109.22 74.93 0)
       (effects (font (size 1.27 1.27)) hide)
@@
       (effects (font (size 1.27 1.27)) (justify left))
     )
-    (property "Value" "" (id 1) (at 229.235 67.31 0)
+    (property "Value" "0.1µF" (id 1) (at 229.235 67.31 0)
       (effects (font (size 1.27 1.27)) (justify left))
     )
-    (property "Footprint" "" (id 2) (at 229.5652 68.58 0)
+    (property "Footprint" "Capacitor_THT:C_Disc_D4.3mm_W1.9mm_P5.00mm" (id 2) (at 229.5652 68.58 0)
       (effects (font (size 1.27 1.27)) hide)
     )
@@
       (effects (font (size 1.27 1.27)) hide)
     )
-    (property "Value" "" (id 1) (at 228.6 54.61 0))
+    (property "Value" "VCC" (id 1) (at 228.6 54.61 0))
     (property "Footprint" "" (id 2) (at 228.6 58.42 0)
       (effects (font (size 1.27 1.27)) hide)
@@
       (effects (font (size 1.27 1.27)) hide)
     )
-    (property "Value" "" (id 1) (at 228.6 74.93 0))
+    (property "Value" "GND" (id 1) (at 228.6 74.93 0))
     (property "Footprint" "" (id 2) (at 228.6 71.12 0)
       (effects (font (size 1.27 1.27)) hide)

Commit message: Fix
Parts:
- D18, D19, D20, D21, D22, D23, D24, D25: symbol Device:LED_ALT -> Device:LED
- U10: symbol 8bit-computer-rescue:74LS245 -> 74xx:74LS245
- U11, U12: symbol 8bit-computer-rescue:74LS173 -> 74xx:74LS173
Connections:
- net B_0: now also D25.2 (A)
- net B_1: now also D24.2 (A)
- net B_2: now also D23.2 (A)
- net B_3: now also D22.2 (A)
- net B_4: now also D21.2 (A)
- net B_5: now also D20.2 (A)
- net B_6: now also D19.2 (A)
- net B_7: now also D18.2 (A)
- net at R32.1: now also D18.1 (K)
- net at R33.1: now also D19.1 (K)
- net at R38.1: now also D24.1 (K)
- net at R34.1: now also D20.1 (K)
- net at R35.1: now also D21.1 (K)
- net at R36.1: now also D22.1 (K)
- net at R37.1: now also D23.1 (K)
- net at R39.1: now also D25.1 (K)
Changed lines of the file:
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@@
     (effects (font (size 1.524 1.524)) (justify left))
   )
-  (symbol (lib_id "8bit-computer-rescue:74LS173") (at 173.99 66.04 270) (unit 1)
+  (symbol (lib_id "74xx:74LS173") (at 173.99 66.04 270) (unit 1)
     (in_bom yes) (on_board yes)
     (property "Reference" "U12" (id 0) (at 176.53 68.58 0))
@@
       (effects (font (size 1.27 1.27)) hide)
     )
-    (property "Datasheet" "" (id 3) (at 173.99 66.04 0)
-      (effects (font (size 1.27 1.27)) hide)
-    )
-  )
-  (symbol (lib_id "8bit-computer-rescue:74LS245") (at 91.44 66.04 90) (unit 1)
+    (property "Datasheet" "http://www.ti.com/lit/gpn/sn74LS173" (id 3) (at 173.99 66.04 0)
+      (effects (font (size 1.27 1.27)) hide)
+    )
+    (pin "1")
+    (pin "10")
+    (pin "11")
+    (pin "12")
+    (pin "13")
+    (pin "14")
+    (pin "15")
+    (pin "16")
+    (pin "2")
+    (pin "3")
+    (pin "4")
+    (pin "5")
+    (pin "6")
+    (pin "7")
+    (pin "8")
+    (pin "9")
+  )
+  (symbol (lib_id "74xx:74LS245") (at 91.44 66.04 90) (unit 1)
     (in_bom yes) (on_board yes)
     (property "Reference" "U10" (id 0) (at 76.835 63.5 0)
@@
       (effects (font (size 1.27 1.27)) hide)
     )
-    (property "Datasheet" "" (id 3) (at 91.44 66.04 0)
-      (effects (font (size 1.27 1.27)) hide)
-    )
-  )
-  (symbol (lib_id "Device:LED_ALT") (at 106.68 139.7 90) (unit 1)
+    (property "Datasheet" "http://www.ti.com/lit/gpn/sn74LS245" (id 3) (at 91.44 66.04 0)
+      (effects (font (size 1.27 1.27)) hide)
+    )
+    (pin "1")
+    (pin "10")
+    (pin "11")
+    (pin "12")
+    (pin "13")
+    (pin "14")
+    (pin "15")
+    (pin "16")
+    (pin "17")
+    (pin "18")
+    (pin "19")
+    (pin "2")
+    (pin "20")
+    (pin "3")
+    (pin "4")
+    (pin "5")
+    (pin "6")
+    (pin "7")
+    (pin "8")
+    (pin "9")
+  )
+  (symbol (lib_id "Device:LED") (at 106.68 139.7 90) (unit 1)
     (in_bom yes) (on_board yes)
     (property "Reference" "D19" (id 0) (at 104.14 139.7 0))
@@
       (effects (font (size 1.27 1.27)) hide)
     )
-    (property "Datasheet" "" (id 3) (at 106.68 139.7 0)
-      (effects (font (size 1.27 1.27)) hide)
-    )
+    (property "Datasheet" "~" (id 3) (at 106.68 139.7 0)
+      (effects (font (size 1.27 1.27)) hide)
+    )
+    (pin "1")
+    (pin "2")
   )
   (symbol (lib_id "Device:R") (at 99.06 151.13 0) (unit 1)
@@
     (pin "1")
   )
-  (symbol (lib_id "8bit-computer-rescue:74LS173") (at 133.35 66.04 270) (unit 1)
+  (symbol (lib_id "74xx:74LS173") (at 133.35 66.04 270) (unit 1)
     (in_bom yes) (on_board yes)
     (property "Reference" "U11" (id 0) (at 135.89 68.58 0))
@@
       (effects (font (size 1.27 1.27)) hide)
     )
-    (property "Datasheet" "" (id 3) (at 133.35 66.04 0)
-      (effects (font (size 1.27 1.27)) hide)
-    )
-  )
-  (symbol (lib_id "Device:LED_ALT") (at 99.06 139.7 90) (unit 1)
+    (property "Datasheet" "http://www.ti.com/lit/gpn/sn74LS173" (id 3) (at 133.35 66.04 0)
+      (effects (font (size 1.27 1.27)) hide)
+    )
+    (pin "1")
+    (pin "10")
+    (pin "11")
+    (pin "12")
+    (pin "13")
+    (pin "14")
+    (pin "15")
+    (pin "16")
+    (pin "2")
+    (pin "3")
+    (pin "4")
+    (pin "5")
+    (pin "6")
+    (pin "7")
+    (pin "8")
+    (pin "9")
+  )
+  (symbol (lib_id "Device:LED") (at 99.06 139.7 90) (unit 1)
     (in_bom yes) (on_board yes)
     (property "Reference" "D18" (id 0) (at 96.52 139.7 0))
@@
       (effects (font (size 1.27 1.27)) hide)
     )
-    (property "Datasheet" "" (id 3) (at 99.06 139.7 0)
-      (effects (font (size 1.27 1.27)) hide)
-    )
-  )
-  (symbol (lib_id "Device:LED_ALT") (at 114.3 139.7 90) (unit 1)
+    (property "Datasheet" "~" (id 3) (at 99.06 139.7 0)
+      (effects (font (size 1.27 1.27)) hide)
+    )
+    (pin "1")
+    (pin "2")
+  )
+  (symbol (lib_id "Device:LED") (at 114.3 139.7 90) (unit 1)
     (in_bom yes) (on_board yes)
     (property "Reference" "D20" (id 0) (at 111.76 139.7 0))
@@
       (effects (font (size 1.27 1.27)) hide)
     )
-    (property "Datasheet" "" (id 3) (at 114.3 139.7 0)
-      (effects (font (size 1.27 1.27)) hide)
-    )
-  )
-  (symbol (lib_id "Device:LED_ALT") (at 121.92 139.7 90) (unit 1)
+    (property "Datasheet" "~" (id 3) (at 114.3 139.7 0)
+      (effects (font (size 1.27 1.27)) hide)
+    )
+    (pin "1")
+    (pin "2")
+  )
+  (symbol (lib_id "Device:LED") (at 121.92 139.7 90) (unit 1)
     (in_bom yes) (on_board yes)
     (property "Reference" "D21" (id 0) (at 119.38 139.7 0))
@@
       (effects (font (size 1.27 1.27)) hide)
     )
-    (property "Datasheet" "" (id 3) (at 121.92 139.7 0)
-      (effects (font (size 1.27 1.27)) hide)
-    )
-  )
-  (symbol (lib_id "Device:LED_ALT") (at 129.54 139.7 90) (unit 1)
+    (property "Datasheet" "~" (id 3) (at 121.92 139.7 0)
+      (effects (font (size 1.27 1.27)) hide)
+    )
+    (pin "1")
+    (pin "2")
+  )
+  (symbol (lib_id "Device:LED") (at 129.54 139.7 90) (unit 1)
     (in_bom yes) (on_board yes)
     (property "Reference" "D22" (id 0) (at 127 139.7 0))
@@
       (effects (font (size 1.27 1.27)) hide)
     )
-    (property "Datasheet" "" (id 3) (at 129.54 139.7 0)
-      (effects (font (size 1.27 1.27)) hide)
-    )
-  )
-  (symbol (lib_id "Device:LED_ALT") (at 137.16 139.7 90) (unit 1)
+    (property "Datasheet" "~" (id 3) (at 129.54 139.7 0)
+      (effects (font (size 1.27 1.27)) hide)
+    )
+    (pin "1")
+    (pin "2")
+  )
+  (symbol (lib_id "Device:LED") (at 137.16 139.7 90) (unit 1)
     (in_bom yes) (on_board yes)
     (property "Reference" "D23" (id 0) (at 134.62 139.7 0))
@@
       (effects (font (size 1.27 1.27)) hide)
     )
-    (property "Datasheet" "" (id 3) (at 137.16 139.7 0)
-      (effects (font (size 1.27 1.27)) hide)
-    )
-  )
-  (symbol (lib_id "Device:LED_ALT") (at 144.78 139.7 90) (unit 1)
+    (property "Datasheet" "~" (id 3) (at 137.16 139.7 0)
+      (effects (font (size 1.27 1.27)) hide)
+    )
+    (pin "1")
+    (pin "2")
+  )
+  (symbol (lib_id "Device:LED") (at 144.78 139.7 90) (unit 1)
     (in_bom yes) (on_board yes)
     (property "Reference" "D24" (id 0) (at 142.24 139.7 0))
@@
       (effects (font (size 1.27 1.27)) hide)
     )
-    (property "Datasheet" "" (id 3) (at 144.78 139.7 0)
-      (effects (font (size 1.27 1.27)) hide)
-    )
-  )
-  (symbol (lib_id "Device:LED_ALT") (at 152.4 139.7 90) (unit 1)
+    (property "Datasheet" "~" (id 3) (at 144.78 139.7 0)
+      (effects (font (size 1.27 1.27)) hide)
+    )
+    (pin "1")
+    (pin "2")
+  )
+  (symbol (lib_id "Device:LED") (at 152.4 139.7 90) (unit 1)
     (in_bom yes) (on_board yes)
     (property "Reference" "D25" (id 0) (at 149.86 139.7 0))
@@
       (effects (font (size 1.27 1.27)) hide)
     )
-    (property "Datasheet" "" (id 3) (at 152.4 139.7 0)
-      (effects (font (size 1.27 1.27)) hide)
-    )
+    (property "Datasheet" "~" (id 3) (at 152.4 139.7 0)
+      (effects (font (size 1.27 1.27)) hide)
+    )
+    (pin "1")
+    (pin "2")
   )
   (symbol (lib_id "Device:R") (at 114.3 151.13 0) (unit 1)
