File: mar.kicad_sch (KiCad schematic)
At the start: 17 parts

Commit message: Fix Clock
Parts:
- C18: value (none) -> 0.1µF; footprint (none) -> Capacitor_THT:C_Disc_D4.3mm_W1.9mm_P5.00mm
- D44, D45, D46, D47: value (none) -> YELLOW; footprint (none) -> LED_THT:LED_D5.0mm
- D48: value (none) -> RED; footprint (none) -> LED_THT:LED_D5.0mm
- D49: value (none) -> GREEN; footprint (none) -> LED_THT:LED_D5.0mm
- R59, R60, R61, R62: value (none) -> 220; footprint (none) -> Resistor_THT:R_Axial_DIN0207_L6.3mm_D2.5mm_P7.62mm_Horizontal
- R63, R64: value (none) -> 1K; footprint (none) -> Resistor_THT:R_Axial_DIN0207_L6.3mm_D2.5mm_P7.62mm_Horizontal
- SW5: value (none) -> SW_DIP_x04; footprint (none) -> Button_Switch_THT:SW_DIP_SPSTx04_Slide_9.78x12.34mm_W7.62mm_P2.54mm
- SW6: value (none) -> SW_SPDT; footprint (none) -> 8bit-custom-footprints:DPDT-pushbutton
- U33: value (none) -> 74LS157; footprint (none) -> Package_DIP:DIP-16_W7.62mm
- U34: value (none) -> 74LS173; footprint (none) -> Package_DIP:DIP-16_W7.62mm
Changed lines of the file:
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@@
     (in_bom yes) (on_board yes)
     (property "Reference" "U33" (id 0) (at 104.14 71.12 0))
-    (property "Value" "" (id 1) (at 111.76 71.12 0))
-    (property "Footprint" "" (id 2) (at 107.95 72.39 0)
+    (property "Value" "74LS157" (id 1) (at 111.76 71.12 0))
+    (property "Footprint" "Package_DIP:DIP-16_W7.62mm" (id 2) (at 107.95 72.39 0)
       (effects (font (size 1.27 1.27)) hide)
     )
@@
     (in_bom yes) (on_board yes)
     (property "Reference" "U34" (id 0) (at 179.07 78.74 0))
-    (property "Value" "" (id 1) (at 175.26 78.74 0))
-    (property "Footprint" "" (id 2) (at 176.53 76.2 0)
+    (property "Value" "74LS173" (id 1) (at 175.26 78.74 0))
+    (property "Footprint" "Package_DIP:DIP-16_W7.62mm" (id 2) (at 176.53 76.2 0)
       (effects (font (size 1.27 1.27)) hide)
     )
@@
     (in_bom yes) (on_board yes)
     (property "Reference" "SW5" (id 0) (at 115.57 119.38 0))
-    (property "Value" "" (id 1) (at 100.33 119.38 0))
-    (property "Footprint" "" (id 2) (at 106.68 119.38 0)
+    (property "Value" "SW_DIP_x04" (id 1) (at 100.33 119.38 0))
+    (property "Footprint" "Button_Switch_THT:SW_DIP_SPSTx04_Slide_9.78x12.34mm_W7.62mm_P2.54mm" (id 2) (at 106.68 119.38 0)
       (effects (font (size 1.27 1.27)) hide)
     )
@@
     (in_bom yes) (on_board yes)
     (property "Reference" "SW6" (id 0) (at 35.56 117.602 0))
-    (property "Value" "" (id 1) (at 35.56 127 0))
-    (property "Footprint" "" (id 2) (at 35.56 121.92 0)
+    (property "Value" "SW_SPDT" (id 1) (at 35.56 127 0))
+    (property "Footprint" "8bit-custom-footprints:DPDT-pushbutton" (id 2) (at 35.56 121.92 0)
       (effects (font (size 1.27 1.27)) hide)
     )
@@
     (in_bom yes) (on_board yes)
     (property "Reference" "D48" (id 0) (at 52.07 115.57 0))
-    (property "Value" "" (id 1) (at 52.07 120.65 0))
-    (property "Footprint" "" (id 2) (at 52.07 118.11 0)
+    (property "Value" "RED" (id 1) (at 52.07 120.65 0))
+    (property "Footprint" "LED_THT:LED_D5.0mm" (id 2) (at 52.07 118.11 0)
       (effects (font (size 1.27 1.27)) hide)
     )
@@
     (in_bom yes) (on_board yes)
     (property "Reference" "D49" (id 0) (at 52.07 123.19 0))
-    (property "Value" "" (id 1) (at 52.07 128.27 0))
-    (property "Footprint" "" (id 2) (at 52.07 125.73 0)
+    (property "Value" "GREEN" (id 1) (at 52.07 128.27 0))
+    (property "Footprint" "LED_THT:LED_D5.0mm" (id 2) (at 52.07 125.73 0)
       (effects (font (size 1.27 1.27)) hide)
     )
@@
     (in_bom yes) (on_board yes)
     (property "Reference" "R63" (id 0) (at 62.992 110.49 90))
-    (property "Value" "" (id 1) (at 60.96 110.49 90))
-    (property "Footprint" "" (id 2) (at 59.182 110.49 90)
+    (property "Value" "1K" (id 1) (at 60.96 110.49 90))
+    (property "Footprint" "Resistor_THT:R_Axial_DIN0207_L6.3mm_D2.5mm_P7.62mm_Horizontal" (id 2) (at 59.182 110.49 90)
       (effects (font (size 1.27 1.27)) hide)
     )
@@
     (in_bom yes) (on_board yes)
     (property "Reference" "R64" (id 0) (at 70.612 110.49 90))
-    (property "Value" "" (id 1) (at 68.58 110.49 90))
-    (property "Footprint" "" (id 2) (at 66.802 110.49 90)
+    (property "Value" "1K" (id 1) (at 68.58 110.49 90))
+    (property "Footprint" "Resistor_THT:R_Axial_DIN0207_L6.3mm_D2.5mm_P7.62mm_Horizontal" (id 2) (at 66.802 110.49 90)
       (effects (font (size 1.27 1.27)) hide)
     )
@@
       (effects (font (size 1.27 1.27)) hide)
     )
-    (property "Value" "" (id 1) (at 27.94 128.27 0))
+    (property "Value" "GND" (id 1) (at 27.94 128.27 0))
     (property "Footprint" "" (id 2) (at 27.94 124.46 0)
       (effects (font (size 1.27 1.27)) hide)
@@
       (effects (font (size 1.27 1.27)) hide)
     )
-    (property "Value" "" (id 1) (at 64.77 97.79 0))
+    (property "Value" "VCC" (id 1) (at 64.77 97.79 0))
     (property "Footprint" "" (id 2) (at 64.77 101.6 0)
       (effects (font (size 1.27 1.27)) hide)
@@
       (effects (font (size 1.27 1.27)) hide)
     )
-    (property "Value" "" (id 1) (at 121.92 135.89 0))
+    (property "Value" "GND" (id 1) (at 121.92 135.89 0))
     (property "Footprint" "" (id 2) (at 121.92 132.08 0)
       (effects (font (size 1.27 1.27)) hide)
@@
     (in_bom yes) (on_board yes)
     (property "Reference" "D47" (id 0) (at 78.74 57.15 0))
-    (property "Value" "" (id 1) (at 83.82 57.15 0))
-    (property "Footprint" "" (id 2) (at 81.28 57.15 0)
+    (property "Value" "YELLOW" (id 1) (at 83.82 57.15 0))
+    (property "Footprint" "LED_THT:LED_D5.0mm" (id 2) (at 81.28 57.15 0)
       (effects (font (size 1.27 1.27)) hide)
     )
@@
     (in_bom yes) (on_board yes)
     (property "Reference" "D46" (id 0) (at 71.12 57.15 0))
-    (property "Value" "" (id 1) (at 76.2 57.15 0))
-    (property "Footprint" "" (id 2) (at 73.66 57.15 0)
+    (property "Value" "YELLOW" (id 1) (at 76.2 57.15 0))
+    (property "Footprint" "LED_THT:LED_D5.0mm" (id 2) (at 73.66 57.15 0)
       (effects (font (size 1.27 1.27)) hide)
     )
@@
     (in_bom yes) (on_board yes)
     (property "Reference" "D45" (id 0) (at 63.5 57.15 0))
-    (property "Value" "" (id 1) (at 68.58 57.15 0))
-    (property "Footprint" "" (id 2) (at 66.04 57.15 0)
+    (property "Value" "YELLOW" (id 1) (at 68.58 57.15 0))
+    (property "Footprint" "LED_THT:LED_D5.0mm" (id 2) (at 66.04 57.15 0)
       (effects (font (size 1.27 1.27)) hide)
     )
@@
     (in_bom yes) (on_board yes)
     (property "Reference" "D44" (id 0) (at 55.88 57.15 0))
-    (property "Value" "" (id 1) (at 60.96 57.15 0))
-    (property "Footprint" "" (id 2) (at 58.42 57.15 0)
+    (property "Value" "YELLOW" (id 1) (at 60.96 57.15 0))
+    (property "Footprint" "LED_THT:LED_D5.0mm" (id 2) (at 58.42 57.15 0)
       (effects (font (size 1.27 1.27)) hide)
     )
@@
     (in_bom yes) (on_board yes)
     (property "Reference" "R62" (id 0) (at 83.312 67.31 90))
-    (property "Value" "" (id 1) (at 81.28 67.31 90))
-    (property "Footprint" "" (id 2) (at 79.502 67.31 90)
+    (property "Value" "220" (id 1) (at 81.28 67.31 90))
+    (property "Footprint" "Resistor_THT:R_Axial_DIN0207_L6.3mm_D2.5mm_P7.62mm_Horizontal" (id 2) (at 79.502 67.31 90)
       (effects (font (size 1.27 1.27)) hide)
     )
@@
     (in_bom yes) (on_board yes)
     (property "Reference" "R61" (id 0) (at 75.692 67.31 90))
-    (property "Value" "" (id 1) (at 73.66 67.31 90))
-    (property "Footprint" "" (id 2) (at 71.882 67.31 90)
+    (property "Value" "220" (id 1) (at 73.66 67.31 90))
+    (property "Footprint" "Resistor_THT:R_Axial_DIN0207_L6.3mm_D2.5mm_P7.62mm_Horizontal" (id 2) (at 71.882 67.31 90)
       (effects (font (size 1.27 1.27)) hide)
     )
@@
     (in_bom yes) (on_board yes)
     (property "Reference" "R60" (id 0) (at 68.072 67.31 90))
-    (property "Value" "" (id 1) (at 66.04 67.31 90))
-    (property "Footprint" "" (id 2) (at 64.262 67.31 90)
+    (property "Value" "220" (id 1) (at 66.04 67.31 90))
+    (property "Footprint" "Resistor_THT:R_Axial_DIN0207_L6.3mm_D2.5mm_P7.62mm_Horizontal" (id 2) (at 64.262 67.31 90)
       (effects (font (size 1.27 1.27)) hide)
     )
@@
     (in_bom yes) (on_board yes)
     (property "Reference" "R59" (id 0) (at 60.452 67.31 90))
-    (property "Value" "" (id 1) (at 58.42 67.31 90))
-    (property "Footprint" "" (id 2) (at 56.642 67.31 90)
+    (property "Value" "220" (id 1) (at 58.42 67.31 90))
+    (property "Footprint" "Resistor_THT:R_Axial_DIN0207_L6.3mm_D2.5mm_P7.62mm_Horizontal" (id 2) (at 56.642 67.31 90)
       (effects (font (size 1.27 1.27)) hide)
     )
@@
       (effects (font (size 1.27 1.27)) hide)
     )
-    (property "Value" "" (id 1) (at 69.85 83.82 0))
+    (property "Value" "GND" (id 1) (at 69.85 83.82 0))
     (property "Footprint" "" (id 2) (at 69.85 80.01 0)
       (effects (font (size 1.27 1.27)) hide)
@@
       (effects (font (size 1.27 1.27)) hide)
     )
-    (property "Value" "" (id 1) (at 175.26 54.61 0))
+    (property "Value" "GND" (id 1) (at 175.26 54.61 0))
     (property "Footprint" "" (id 2) (at 175.26 50.8 0)
       (effects (font (size 1.27 1.27)) hide)
@@
       (effects (font (size 1.27 1.27)) (justify left))
     )
-    (property "Value" "" (id 1) (at 219.075 82.55 0)
+    (property "Value" "0.1µF" (id 1) (at 219.075 82.55 0)
       (effects (font (size 1.27 1.27)) (justify left))
     )
-    (property "Footprint" "" (id 2) (at 219.4052 83.82 0)
+    (property "Footprint" "Capacitor_THT:C_Disc_D4.3mm_W1.9mm_P5.00mm" (id 2) (at 219.4052 83.82 0)
       (effects (font (size 1.27 1.27)) hide)
     )
@@
       (effects (font (size 1.27 1.27)) hide)
     )
-    (property "Value" "" (id 1) (at 218.44 69.85 0))
+    (property "Value" "VCC" (id 1) (at 218.44 69.85 0))
     (property "Footprint" "" (id 2) (at 218.44 73.66 0)
       (effects (font (size 1.27 1.27)) hide)
@@
       (effects (font (size 1.27 1.27)) hide)
     )
-    (property "Value" "" (id 1) (at 218.44 90.17 0))
+    (property "Value" "GND" (id 1) (at 218.44 90.17 0))
     (property "Footprint" "" (id 2) (at 218.44 86.36 0)
       (effects (font (size 1.27 1.27)) hide)

Commit message: Fix
Parts:
- D44, D45, D46, D47, D48, D49: symbol Device:LED_ALT -> Device:LED
- SW5: symbol 8bit-computer-rescue:SW_DIP_x04 -> Switch:SW_DIP_x04
- SW6: symbol 8bit-computer-rescue:SW_SPDT -> Switch:SW_SPDT
- U33: symbol 8bit-computer-rescue:74LS157 -> 74xx:74LS157
- U34: symbol 8bit-computer-rescue:74LS173 -> 74xx:74LS173
Connections:
- net A0: now also D47.2 (A), U33.12 (Zd)
- net A1: now also D46.2 (A), U33.9 (Zc)
- net A2: now also D45.2 (A), U33.7 (Zb)
- net A3: now also D44.2 (A), U33.4 (Za)
- net BUS_0: now also U34.11 (D3)
- net BUS_1: now also U34.12 (D2)
- net BUS_2: now also U34.13 (D1)
- net BUS_3: now also U34.14 (D0)
- net CLK: now also U34.7 (Cp)
- net CLR: now also U34.15 (Mr)
- net GND: now also SW5.3, SW5.4, SW5.7, SW5.8, SW6.2 (B), U33.15 (E), U34.1 (Oe1), U34.2 (Oe2)
- net PROG: now also D48.1 (K), SW6.1 (A), U33.1 (S)
- net ~{MI}: now also U34.10 (E2), U34.9 (E1)
- net at R63.2: now also D48.2 (A)
- net at R64.2: now also D49.2 (A)
- net at R62.1: now also D47.1 (K)
- net at R61.1: now also D46.1 (K)
- net at R60.1: now also D45.1 (K)
- net at R59.1: now also D44.1 (K)
- new net: U33.10 (I1c), U34.5 (Q2)
- new net: SW5.2, U33.11 (I0c)
- new net: U33.13 (I1d), U34.6 (Q3)
- new net: SW5.1, U33.14 (I0d)
- new net: SW5.5, U33.2 (I0a)
- new net: U33.3 (I1a), U34.3 (Q0)
- new net: SW5.6, U33.5 (I0b)
- new net: U33.6 (I1b), U34.4 (Q1)
- new net: D49.1 (K), SW6.3 (C)
