File: output.kicad_sch (KiCad schematic)
At the start: 18 parts

Commit message: Fix Clock
Parts:
- C20, C21: value (none) -> 0.1µF; footprint (none) -> Capacitor_THT:C_Disc_D4.3mm_W1.9mm_P5.00mm
- C8, C9: value (none) -> 0.01µF; footprint (none) -> Capacitor_THT:C_Disc_D4.3mm_W1.9mm_P5.00mm
- R104: value (none) -> 10k; footprint (none) -> Resistor_THT:R_Axial_DIN0207_L6.3mm_D2.5mm_P7.62mm_Horizontal
- R65: value (none) -> 1K; footprint (none) -> Resistor_THT:R_Axial_DIN0207_L6.3mm_D2.5mm_P7.62mm_Horizontal
- R66: value (none) -> 100K; footprint (none) -> Resistor_THT:R_Axial_DIN0207_L6.3mm_D2.5mm_P7.62mm_Horizontal
- SW7: value (none) -> SW_SPDT; footprint (none) -> 8bit-custom-footprints:DPDT-pushbutton
- U37: value (none) -> 74LS76; footprint (none) -> Package_DIP:DIP-16_W7.62mm
- U38: value (none) -> 74LS139; footprint (none) -> Package_DIP:DIP-16_W7.62mm
- U39: value (none) -> LM555; footprint (none) -> Package_DIP:DIP-8_W7.62mm; symbol 8bit-computer-rescue:LM555 -> Timer:LM555xN
- U40, U41, U42, U43: value (none) -> 7SEGMENT_CC; footprint (none) -> Display_7Segment:7SegmentLED_LTS6760_LTS6780
- U44: value (none) -> 74LS273; footprint (none) -> Package_DIP:DIP-20_W7.62mm
- U45: value (none) -> 28C16; footprint (none) -> Package_DIP:DIP-24_W15.24mm_Socket
- U46: value (none) -> 74LS08; footprint (none) -> Package_DIP:DIP-14_W7.62mm; symbol 8bit-computer-rescue:74LS08 -> 74xx:74LS08
Connections:
- net GND: now also U39.1 (GND)
- net VCC: now also U39.8 (VCC)
- net at R65.2, R66.1: now also U39.7 (DIS)
- net at C8.1, R66.2: now also U39.2 (TR), U39.6 (THR)
- net at C9.1: now also U39.5 (CV)

Commit message: Fix
Parts:
- SW7: symbol 8bit-computer-rescue:SW_SPDT -> Switch:SW_SPDT
Connections:
- net VCC: now also SW7.3 (C)
- net at R104.1: now also SW7.1 (A)
Changed lines of the file:
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@@
     (pin "1")
   )
-  (symbol (lib_id "8bit-computer-rescue:SW_SPDT") (at 45.72 144.78 180) (unit 1)
+  (symbol (lib_id "Switch:SW_SPDT") (at 45.72 144.78 180) (unit 1)
     (in_bom yes) (on_board yes)
     (property "Reference" "SW7" (id 0) (at 45.72 149.098 0))
@@
       (effects (font (size 1.27 1.27)) hide)
     )
-    (property "Datasheet" "" (id 3) (at 45.72 144.78 0)
+    (property "Datasheet" "~" (id 3) (at 45.72 144.78 0)
       (effects (font (size 1.27 1.27)) hide)
     )
+    (pin "1")
+    (pin "2")
+    (pin "3")
   )
   (symbol (lib_id "power:VCC") (at 38.1 139.7 0) (unit 1)
