File: program-counter.kicad_sch (KiCad schematic)
At the start: 11 parts

Commit message: Fix Clock
Parts:
- C19: value (none) -> 0.1µF; footprint (none) -> Capacitor_THT:C_Disc_D4.3mm_W1.9mm_P5.00mm
- D82, D83, D84, D85: value (none) -> GREEN; footprint (none) -> LED_THT:LED_D5.0mm
- R100, R101, R102, R103: value (none) -> 220; footprint (none) -> Resistor_THT:R_Axial_DIN0207_L6.3mm_D2.5mm_P7.62mm_Horizontal
- U35: value (none) -> 74LS161; footprint (none) -> Package_DIP:DIP-16_W7.62mm
- U36: value (none) -> 74LS245; footprint (none) -> Package_DIP:DIP-20_W7.62mm
Changed lines of the file:
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@@
     (in_bom yes) (on_board yes)
     (property "Reference" "U35" (id 0) (at 138.43 63.5 0))
-    (property "Value" "" (id 1) (at 137.16 55.88 0))
-    (property "Footprint" "" (id 2) (at 139.7 60.96 0)
+    (property "Value" "74LS161" (id 1) (at 137.16 55.88 0))
+    (property "Footprint" "Package_DIP:DIP-16_W7.62mm" (id 2) (at 139.7 60.96 0)
       (effects (font (size 1.27 1.27)) hide)
     )
@@
       (effects (font (size 1.27 1.27)) (justify left bottom))
     )
-    (property "Value" "" (id 1) (at 82.55 83.185 0)
+    (property "Value" "74LS245" (id 1) (at 82.55 83.185 0)
       (effects (font (size 1.27 1.27)) (justify left top))
     )
-    (property "Footprint" "" (id 2) (at 81.28 68.58 0)
+    (property "Footprint" "Package_DIP:DIP-20_W7.62mm" (id 2) (at 81.28 68.58 0)
       (effects (font (size 1.27 1.27)) hide)
     )
@@
       (effects (font (size 1.27 1.27)) hide)
     )
-    (property "Value" "" (id 1) (at 57.15 91.44 0))
+    (property "Value" "GND" (id 1) (at 57.15 91.44 0))
     (property "Footprint" "" (id 2) (at 57.15 87.63 0)
       (effects (font (size 1.27 1.27)) hide)
@@
       (effects (font (size 1.27 1.27)) (justify left))
     )
-    (property "Value" "" (id 1) (at 208.915 74.93 0)
+    (property "Value" "0.1µF" (id 1) (at 208.915 74.93 0)
       (effects (font (size 1.27 1.27)) (justify left))
     )
-    (property "Footprint" "" (id 2) (at 209.2452 76.2 0)
+    (property "Footprint" "Capacitor_THT:C_Disc_D4.3mm_W1.9mm_P5.00mm" (id 2) (at 209.2452 76.2 0)
       (effects (font (size 1.27 1.27)) hide)
     )
@@
       (effects (font (size 1.27 1.27)) hide)
     )
-    (property "Value" "" (id 1) (at 208.28 82.55 0))
+    (property "Value" "GND" (id 1) (at 208.28 82.55 0))
     (property "Footprint" "" (id 2) (at 208.28 78.74 0)
       (effects (font (size 1.27 1.27)) hide)
@@
       (effects (font (size 1.27 1.27)) hide)
     )
-    (property "Value" "" (id 1) (at 208.28 62.23 0))
+    (property "Value" "VCC" (id 1) (at 208.28 62.23 0))
     (property "Footprint" "" (id 2) (at 208.28 66.04 0)
       (effects (font (size 1.27 1.27)) hide)
@@
     (in_bom yes) (on_board yes)
     (property "Reference" "D82" (id 0) (at 104.14 36.83 0))
-    (property "Value" "" (id 1) (at 99.06 36.83 0))
-    (property "Footprint" "" (id 2) (at 101.6 36.83 0)
+    (property "Value" "GREEN" (id 1) (at 99.06 36.83 0))
+    (property "Footprint" "LED_THT:LED_D5.0mm" (id 2) (at 101.6 36.83 0)
       (effects (font (size 1.27 1.27)) hide)
     )
@@
     (in_bom yes) (on_board yes)
     (property "Reference" "D83" (id 0) (at 109.22 36.83 0))
-    (property "Value" "" (id 1) (at 104.14 36.83 0))
-    (property "Footprint" "" (id 2) (at 106.68 36.83 0)
+    (property "Value" "GREEN" (id 1) (at 104.14 36.83 0))
+    (property "Footprint" "LED_THT:LED_D5.0mm" (id 2) (at 106.68 36.83 0)
       (effects (font (size 1.27 1.27)) hide)
     )
@@
     (in_bom yes) (on_board yes)
     (property "Reference" "D84" (id 0) (at 114.3 36.83 0))
-    (property "Value" "" (id 1) (at 109.22 36.83 0))
-    (property "Footprint" "" (id 2) (at 111.76 36.83 0)
+    (property "Value" "GREEN" (id 1) (at 109.22 36.83 0))
+    (property "Footprint" "LED_THT:LED_D5.0mm" (id 2) (at 111.76 36.83 0)
       (effects (font (size 1.27 1.27)) hide)
     )
@@
     (in_bom yes) (on_board yes)
     (property "Reference" "D85" (id 0) (at 119.38 36.83 0))
-    (property "Value" "" (id 1) (at 114.3 36.83 0))
-    (property "Footprint" "" (id 2) (at 116.84 36.83 0)
+    (property "Value" "GREEN" (id 1) (at 114.3 36.83 0))
+    (property "Footprint" "LED_THT:LED_D5.0mm" (id 2) (at 116.84 36.83 0)
       (effects (font (size 1.27 1.27)) hide)
     )
@@
     (in_bom yes) (on_board yes)
     (property "Reference" "R100" (id 0) (at 103.632 26.67 90))
-    (property "Value" "" (id 1) (at 101.6 26.67 90))
-    (property "Footprint" "" (id 2) (at 99.822 26.67 90)
+    (property "Value" "220" (id 1) (at 101.6 26.67 90))
+    (property "Footprint" "Resistor_THT:R_Axial_DIN0207_L6.3mm_D2.5mm_P7.62mm_Horizontal" (id 2) (at 99.822 26.67 90)
       (effects (font (size 1.27 1.27)) hide)
     )
@@
     (in_bom yes) (on_board yes)
     (property "Reference" "R101" (id 0) (at 108.712 26.67 90))
-    (property "Value" "" (id 1) (at 106.68 26.67 90))
-    (property "Footprint" "" (id 2) (at 104.902 26.67 90)
+    (property "Value" "220" (id 1) (at 106.68 26.67 90))
+    (property "Footprint" "Resistor_THT:R_Axial_DIN0207_L6.3mm_D2.5mm_P7.62mm_Horizontal" (id 2) (at 104.902 26.67 90)
       (effects (font (size 1.27 1.27)) hide)
     )
@@
     (in_bom yes) (on_board yes)
     (property "Reference" "R102" (id 0) (at 113.792 26.67 90))
-    (property "Value" "" (id 1) (at 111.76 26.67 90))
-    (property "Footprint" "" (id 2) (at 109.982 26.67 90)
+    (property "Value" "220" (id 1) (at 111.76 26.67 90))
+    (property "Footprint" "Resistor_THT:R_Axial_DIN0207_L6.3mm_D2.5mm_P7.62mm_Horizontal" (id 2) (at 109.982 26.67 90)
       (effects (font (size 1.27 1.27)) hide)
     )
@@
     (in_bom yes) (on_board yes)
     (property "Reference" "R103" (id 0) (at 118.872 26.67 90))
-    (property "Value" "" (id 1) (at 116.84 26.67 90))
-    (property "Footprint" "" (id 2) (at 115.062 26.67 90)
+    (property "Value" "220" (id 1) (at 116.84 26.67 90))
+    (property "Footprint" "Resistor_THT:R_Axial_DIN0207_L6.3mm_D2.5mm_P7.62mm_Horizontal" (id 2) (at 115.062 26.67 90)
       (effects (font (size 1.27 1.27)) hide)
     )
@@
       (effects (font (size 1.27 1.27)) hide)
     )
-    (property "Value" "" (id 1) (at 124.46 29.21 0))
+    (property "Value" "GND" (id 1) (at 124.46 29.21 0))
     (property "Footprint" "" (id 2) (at 124.46 25.4 0)
       (effects (font (size 1.27 1.27)) hide)

Commit message: Fix
Parts:
- D82, D83, D84, D85: symbol Device:LED_ALT -> Device:LED
- U35: symbol 8bit-computer-rescue:74LS161 -> 74xx:74LS161
- U36: symbol 8bit-computer-rescue:74LS245 -> 74xx:74LS245
Connections:
- net BUS_0: now also U35.6 (D3), U36.9 (A7)
- net BUS_1: now also U35.5 (D2), U36.8 (A6)
- net BUS_2: now also U35.4 (D1), U36.7 (A5)
- net BUS_3: now also U35.3 (D0), U36.6 (A4)
- net CE: now also U35.10 (CET), U35.7 (CEP)
- net CLK: now also U35.2 (CP)
- net GND: now also U36.1 (A->B)
- net ~{CLR}: now also U35.1 (~{MR})
- net ~{CO}: now also U36.19 (CE)
- net ~{J}: now also U35.9 (~{PE})
- net at R100.2: now also D82.1 (K)
- net at R101.2: now also D83.1 (K)
- net at R102.2: now also D84.1 (K)
- net at R103.2: now also D85.1 (K)
- new net: D82.2 (A), U35.11 (Q3), U36.14 (B4)
- new net: D83.2 (A), U35.12 (Q2), U36.13 (B5)
- new net: D84.2 (A), U35.13 (Q1), U36.12 (B6)
- new net: D85.2 (A), U35.14 (Q0), U36.11 (B7)
- no-connect marks 9 -> 0
