File: ram.kicad_sch (KiCad schematic)
At the start: 31 parts

Commit message: Fix Clock
Parts:
- C16, C17: value (none) -> 0.1µF; footprint (none) -> Capacitor_THT:C_Disc_D4.3mm_W1.9mm_P5.00mm
- C7: value (none) -> 0.01µF; footprint (none) -> Capacitor_THT:C_Disc_D4.3mm_W1.9mm_P5.00mm
- D36, D37, D38, D39, D40, D41, D42, D43: value (none) -> RED; footprint (none) -> LED_THT:LED_D5.0mm
- R50, R51, R52, R53, R54, R55, R56, R57: value (none) -> 220; footprint (none) -> Resistor_THT:R_Axial_DIN0207_L6.3mm_D2.5mm_P7.62mm_Horizontal
- R58: value (none) -> 1K; footprint (none) -> Resistor_THT:R_Axial_DIN0207_L6.3mm_D2.5mm_P7.62mm_Horizontal
- SW3: value (none) -> SW_DIP_x08; footprint (none) -> Button_Switch_THT:SW_DIP_SPSTx08_Slide_9.78x22.5mm_W7.62mm_P2.54mm
- SW4: value (none) -> SW_Push; footprint (none) -> Button_Switch_THT:SW_PUSH_6mm_H5mm
- U24, U25: value (none) -> 74189; footprint (none) -> Package_DIP:DIP-16_W7.62mm
- U26, U27, U32: value (none) -> 74LS157; footprint (none) -> Package_DIP:DIP-16_W7.62mm
- U28, U29: value (none) -> 74LS04; footprint (none) -> Package_DIP:DIP-14_W7.62mm; symbol 8bit-computer-rescue:74LS04 -> 74xx:74LS04
- U30: value (none) -> 74LS245; footprint (none) -> Package_DIP:DIP-20_W7.62mm
- U31: value (none) -> 74LS00; footprint (none) -> Package_DIP:DIP-14_W7.62mm

Commit message: Fix
Parts:
- D36, D37, D38, D39, D40, D41, D42, D43: symbol Device:LED_ALT -> Device:LED
- SW3: symbol 8bit-computer-rescue:SW_DIP_x08 -> Switch:SW_DIP_x08
- SW4: symbol 8bit-computer-rescue:SW_Push -> Switch:SW_Push
- U26, U27, U32: symbol 8bit-computer-rescue:74LS157 -> 74xx:74LS157
- U30: symbol 8bit-computer-rescue:74LS245 -> 74xx:74LS245
- U31: symbol 8bit-computer-rescue:74LS00 -> 74xx:74LS00
Connections:
- net BUS_0: now also U27.13 (I1d), U30.11 (B7)
- net BUS_1: now also U27.10 (I1c), U30.12 (B6)
- net BUS_2: now also U27.6 (I1b), U30.13 (B5)
- net BUS_3: now also U27.3 (I1a), U30.14 (B4)
- net BUS_4: now also U26.13 (I1d), U30.15 (B3)
- net BUS_5: now also U26.10 (I1c), U30.16 (B2)
- net BUS_6: now also U26.6 (I1b), U30.17 (B1)
- net BUS_7: now also U26.3 (I1a), U30.18 (B0)
- net GND: now also SW3.11, SW3.12, SW3.15, SW3.16, SW3.3, SW3.4, SW3.7, SW3.8, SW4.1, U26.15 (E), U27.15 (E), U32.15 (E)
- net PROG: now also U26.1 (S), U27.1 (S), U32.1 (S)
- net RI: now also U31.2
- net VCC: now also U30.1 (A->B)
- net ~{RO}: now also U30.19 (CE)
- net at U28.2: now also D36.2 (A), U30.2 (A0)
- net at U28.4: now also D37.2 (A), U30.3 (A1)
- net at U28.6: now also D38.2 (A), U30.4 (A2)
- net at U28.8: now also D39.2 (A), U30.5 (A3)
- net at U29.6: now also D43.2 (A), U30.9 (A7)
- net at U29.4: now also D42.2 (A), U30.8 (A6)
- net at U29.2: now also D41.2 (A), U30.7 (A5)
- net at U29.12: now also D40.2 (A), U30.6 (A4)
- net at C7.2, R58.2: now also U31.1
- net at R50.1: now also D36.1 (K)
- net at R51.1: now also D37.1 (K)
- net at R52.1: now also D38.1 (K)
- net at R53.1: now also D39.1 (K)
- net at R54.1: now also D40.1 (K)
- net at R55.1: now also D41.1 (K)
- net at R56.1: now also D42.1 (K)
- net at R57.1: now also D43.1 (K)
- new net: SW3.6, U26.11 (I0c)
- new net: SW3.5, U26.14 (I0d)
- new net: SW3.9, U26.2 (I0a)
- new net: SW3.10, U26.5 (I0b)
- new net: SW3.2, U27.11 (I0c)
- new net: SW3.1, U27.14 (I0d)
- new net: SW3.13, U27.2 (I0a)
- new net: SW3.14, U27.5 (I0b)
- new net: U31.3, U32.10 (I1c)
- new net: SW4.2, U32.11 (I0c)
