File: 8bit-computer.kicad_sch (KiCad schematic)
At the start: 26 parts

Commit message: Fix Clock
Parts:
- C24: value (none) -> 10µF; footprint (none) -> Capacitor_THT:CP_Radial_D5.0mm_P2.00mm
- D2, D3, D4, D5, D6, D7, D8, D9: value (none) -> RED; footprint (none) -> LED_THT:LED_D5.0mm
- J1: value (none) -> USB_B; footprint (none) -> Connector_USB:USB_B_OST_USB-B1HSxx_Horizontal
- R10, R11, R12, R13, R14, R15, R8, R9: value (none) -> 10K; footprint (none) -> Resistor_THT:R_Axial_DIN0207_L6.3mm_D2.5mm_P7.62mm_Horizontal
- R16, R17, R18, R19, R20, R21, R22, R23: value (none) -> 220; footprint (none) -> Resistor_THT:R_Axial_DIN0207_L6.3mm_D2.5mm_P7.62mm_Horizontal

Commit message: Fix
Parts:
- D2, D3, D4, D5, D6, D7, D8, D9: symbol Device:LED_ALT -> Device:LED
Connections:
- net A register/BUS_0: now also D9.2 (A)
- net A register/BUS_1: now also D8.2 (A)
- net A register/BUS_2: now also D7.2 (A)
- net A register/BUS_3: now also D6.2 (A)
- net A register/BUS_4: now also D5.2 (A)
- net A register/BUS_5: now also D4.2 (A)
- net A register/BUS_6: now also D3.2 (A)
- net A register/BUS_7: now also D2.2 (A)
- net at R16.1: now also D2.1 (K)
- net at R17.1: now also D3.1 (K)
- net at R18.1: now also D4.1 (K)
- net at R19.1: now also D5.1 (K)
- net at R20.1: now also D6.1 (K)
- net at R21.1: now also D7.1 (K)
- net at R22.1: now also D8.1 (K)
- net at R23.1: now also D9.1 (K)
Changed lines of the file:
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@@
     (pin "1")
   )
-  (symbol (lib_id "Device:LED_ALT") (at 88.9 237.49 90) (unit 1)
+  (symbol (lib_id "Device:LED") (at 88.9 237.49 90) (unit 1)
     (in_bom yes) (on_board yes)
     (property "Reference" "D9" (id 0) (at 86.36 237.49 0))
@@
       (effects (font (size 1.27 1.27)) hide)
     )
-    (property "Datasheet" "" (id 3) (at 88.9 237.49 0)
+    (property "Datasheet" "~" (id 3) (at 88.9 237.49 0)
       (effects (font (size 1.27 1.27)) hide)
     )
+    (pin "1")
+    (pin "2")
   )
-  (symbol (lib_id "Device:LED_ALT") (at 83.82 237.49 90) (unit 1)
+  (symbol (lib_id "Device:LED") (at 83.82 237.49 90) (unit 1)
     (in_bom yes) (on_board yes)
     (property "Reference" "D8" (id 0) (at 81.28 237.49 0))
@@
       (effects (font (size 1.27 1.27)) hide)
     )
-    (property "Datasheet" "" (id 3) (at 83.82 237.49 0)
+    (property "Datasheet" "~" (id 3) (at 83.82 237.49 0)
       (effects (font (size 1.27 1.27)) hide)
     )
+    (pin "1")
+    (pin "2")
   )
-  (symbol (lib_id "Device:LED_ALT") (at 78.74 237.49 90) (unit 1)
+  (symbol (lib_id "Device:LED") (at 78.74 237.49 90) (unit 1)
     (in_bom yes) (on_board yes)
     (property "Reference" "D7" (id 0) (at 76.2 237.49 0))
@@
       (effects (font (size 1.27 1.27)) hide)
     )
-    (property "Datasheet" "" (id 3) (at 78.74 237.49 0)
+    (property "Datasheet" "~" (id 3) (at 78.74 237.49 0)
       (effects (font (size 1.27 1.27)) hide)
     )
+    (pin "1")
+    (pin "2")
   )
-  (symbol (lib_id "Device:LED_ALT") (at 73.66 237.49 90) (unit 1)
+  (symbol (lib_id "Device:LED") (at 73.66 237.49 90) (unit 1)
     (in_bom yes) (on_board yes)
     (property "Reference" "D6" (id 0) (at 71.12 237.49 0))
@@
       (effects (font (size 1.27 1.27)) hide)
     )
-    (property "Datasheet" "" (id 3) (at 73.66 237.49 0)
+    (property "Datasheet" "~" (id 3) (at 73.66 237.49 0)
       (effects (font (size 1.27 1.27)) hide)
     )
+    (pin "1")
+    (pin "2")
   )
-  (symbol (lib_id "Device:LED_ALT") (at 68.58 237.49 90) (unit 1)
+  (symbol (lib_id "Device:LED") (at 68.58 237.49 90) (unit 1)
     (in_bom yes) (on_board yes)
     (property "Reference" "D5" (id 0) (at 66.04 237.49 0))
@@
       (effects (font (size 1.27 1.27)) hide)
     )
-    (property "Datasheet" "" (id 3) (at 68.58 237.49 0)
+    (property "Datasheet" "~" (id 3) (at 68.58 237.49 0)
       (effects (font (size 1.27 1.27)) hide)
     )
+    (pin "1")
+    (pin "2")
   )
-  (symbol (lib_id "Device:LED_ALT") (at 63.5 237.49 90) (unit 1)
+  (symbol (lib_id "Device:LED") (at 63.5 237.49 90) (unit 1)
     (in_bom yes) (on_board yes)
     (property "Reference" "D4" (id 0) (at 60.96 237.49 0))
@@
       (effects (font (size 1.27 1.27)) hide)
     )
-    (property "Datasheet" "" (id 3) (at 63.5 237.49 0)
+    (property "Datasheet" "~" (id 3) (at 63.5 237.49 0)
       (effects (font (size 1.27 1.27)) hide)
     )
+    (pin "1")
+    (pin "2")
   )
-  (symbol (lib_id "Device:LED_ALT") (at 58.42 237.49 90) (unit 1)
+  (symbol (lib_id "Device:LED") (at 58.42 237.49 90) (unit 1)
     (in_bom yes) (on_board yes)
     (property "Reference" "D3" (id 0) (at 55.88 237.49 0))
@@
       (effects (font (size 1.27 1.27)) hide)
     )
-    (property "Datasheet" "" (id 3) (at 58.42 237.49 0)
+    (property "Datasheet" "~" (id 3) (at 58.42 237.49 0)
       (effects (font (size 1.27 1.27)) hide)
     )
+    (pin "1")
+    (pin "2")
   )
-  (symbol (lib_id "Device:LED_ALT") (at 53.34 237.49 90) (unit 1)
+  (symbol (lib_id "Device:LED") (at 53.34 237.49 90) (unit 1)
     (in_bom yes) (on_board yes)
     (property "Reference" "D2" (id 0) (at 50.8 237.49 0))
@@
       (effects (font (size 1.27 1.27)) hide)
     )
-    (property "Datasheet" "" (id 3) (at 53.34 237.49 0)
+    (property "Datasheet" "~" (id 3) (at 53.34 237.49 0)
       (effects (font (size 1.27 1.27)) hide)
     )
+    (pin "1")
+    (pin "2")
   )
   (symbol (lib_id "Device:R") (at 53.34 247.65 0) (unit 1)

Commit message: Fix ALU
Parts:
- C24: symbol Device:CP1 -> Device:C
- J1: symbol 8bit-computer-rescue:USB_B -> Connector:USB_B
Connections:
- net GND: now also C24.2, J1.4 (GND), J1.5 (Shield)
- net VCC: now also C24.1, J1.1 (VBUS)
Changed lines of the file:
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@@
     (pin "2")
   )
-  (symbol (lib_id "8bit-computer-rescue:USB_B") (at 170.18 210.82 0) (unit 1)
+  (symbol (lib_id "Connector:USB_B") (at 170.18 210.82 0) (unit 1)
     (in_bom yes) (on_board yes)
     (property "Reference" "J1" (id 0) (at 165.1 199.39 0)
@@
       (effects (font (size 1.27 1.27)) hide)
     )
-    (property "Datasheet" "" (id 3) (at 173.99 212.09 0)
+    (property "Datasheet" " ~" (id 3) (at 173.99 212.09 0)
       (effects (font (size 1.27 1.27)) hide)
     )
+    (pin "1")
+    (pin "2")
+    (pin "3")
+    (pin "4")
+    (pin "5")
   )
-  (symbol (lib_id "Device:CP1") (at 185.42 219.71 0) (unit 1)
+  (symbol (lib_id "Device:C") (at 185.42 219.71 0) (unit 1)
     (in_bom yes) (on_board yes)
     (property "Reference" "C24" (id 0) (at 186.055 217.17 0)
@@
       (effects (font (size 1.27 1.27)) (justify left))
     )
-    (property "Footprint" "Capacitor_THT:CP_Radial_D5.0mm_P2.00mm" (id 2) (at 185.42 219.71 0)
+    (property "Footprint" "Capacitor_THT:CP_Radial_D5.0mm_P2.00mm" (id 2) (at 186.3852 223.52 0)
       (effects (font (size 1.27 1.27)) hide)
     )
-    (property "Datasheet" "" (id 3) (at 185.42 219.71 0)
+    (property "Datasheet" "~" (id 3) (at 185.42 219.71 0)
       (effects (font (size 1.27 1.27)) hide)
     )
+    (pin "1")
+    (pin "2")
   )
   (sheet (at 60.96 20.32) (size 17.78 11.43) (fields_autoplaced)
