File: alu.kicad_sch (KiCad schematic)
At the start: 30 parts

Commit message: Fix Clock
Parts:
- C14, C15: value (none) -> 0.1µF; footprint (none) -> Capacitor_THT:C_Disc_D4.3mm_W1.9mm_P5.00mm
- D34, D35: value (none) -> GREEN; footprint (none) -> LED_THT:LED_D5.0mm
- D74, D75, D76, D77, D78, D79, D80, D81: value (none) -> RED; footprint (none) -> LED_THT:LED_D5.0mm
- R48, R49, R92, R93, R94, R95, R96, R97, R98, R99: value (none) -> 220; footprint (none) -> Resistor_THT:R_Axial_DIN0207_L6.3mm_D2.5mm_P7.62mm_Horizontal
- U16, U18: value (none) -> 74LS86; footprint (none) -> Package_DIP:DIP-14_W7.62mm
- U17: value (none) -> 74LS245; footprint (none) -> Package_DIP:DIP-20_W7.62mm
- U19: value (none) -> 74LS173; footprint (none) -> Package_DIP:DIP-16_W7.62mm
- U20, U21: value (none) -> 74LS283; footprint (none) -> Package_DIP:DIP-16_W7.62mm
- U22: value (none) -> 74LS02; footprint (none) -> Package_DIP:DIP-14_W7.62mm
- U23: value (none) -> 74LS08; footprint (none) -> Package_DIP:DIP-14_W7.62mm; symbol 8bit-computer-rescue:74LS08 -> 74xx:74LS08

Commit message: Fix
Parts:
- D34, D35, D74, D75, D76, D77, D78, D79, D80, D81: symbol Device:LED_ALT -> Device:LED
- U17: symbol 8bit-computer-rescue:74LS245 -> 74xx:74LS245
- U19: symbol 8bit-computer-rescue:74LS173 -> 74xx:74LS173
Connections:
- net CF: now also D34.2 (A)
- net ZF: now also D35.2 (A)
- net at R48.2: now also D34.1 (K)
- net at R49.2: now also D35.1 (K)
- net at R92.1: now also D74.1 (K)
- net at R93.1: now also D75.1 (K)
- net at R94.1: now also D76.1 (K)
- net at R95.1: now also D77.1 (K)
- net at R96.1: now also D78.1 (K)
- net at R97.1: now also D79.1 (K)
- net at R98.1: now also D80.1 (K)
- net at R99.1: now also D81.1 (K)
Changed lines of the file:
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@@
     (effects (font (size 1.524 1.524)) (justify left))
   )
-  (symbol (lib_id "8bit-computer-rescue:74LS245") (at 118.11 58.42 90) (unit 1)
+  (symbol (lib_id "74xx:74LS245") (at 118.11 58.42 90) (unit 1)
     (in_bom yes) (on_board yes)
     (property "Reference" "U17" (id 0) (at 103.505 55.88 0)
@@
       (effects (font (size 1.27 1.27)) hide)
     )
-    (property "Datasheet" "" (id 3) (at 118.11 58.42 0)
-      (effects (font (size 1.27 1.27)) hide)
-    )
+    (property "Datasheet" "http://www.ti.com/lit/gpn/sn74LS245" (id 3) (at 118.11 58.42 0)
+      (effects (font (size 1.27 1.27)) hide)
+    )
+    (pin "1")
+    (pin "10")
+    (pin "11")
+    (pin "12")
+    (pin "13")
+    (pin "14")
+    (pin "15")
+    (pin "16")
+    (pin "17")
+    (pin "18")
+    (pin "19")
+    (pin "2")
+    (pin "20")
+    (pin "3")
+    (pin "4")
+    (pin "5")
+    (pin "6")
+    (pin "7")
+    (pin "8")
+    (pin "9")
   )
   (symbol (lib_id "8bit-computer-rescue:74LS283") (at 153.67 93.98 180) (unit 1)
@@
     (pin "7")
   )
-  (symbol (lib_id "8bit-computer-rescue:74LS173") (at 46.99 88.9 90) (unit 1)
+  (symbol (lib_id "74xx:74LS173") (at 46.99 88.9 90) (unit 1)
     (in_bom yes) (on_board yes)
     (property "Reference" "U19" (id 0) (at 44.45 86.36 0))
@@
       (effects (font (size 1.27 1.27)) hide)
     )
-    (property "Datasheet" "" (id 3) (at 46.99 88.9 0)
-      (effects (font (size 1.27 1.27)) hide)
-    )
+    (property "Datasheet" "http://www.ti.com/lit/gpn/sn74LS173" (id 3) (at 46.99 88.9 0)
+      (effects (font (size 1.27 1.27)) hide)
+    )
+    (pin "1")
+    (pin "10")
+    (pin "11")
+    (pin "12")
+    (pin "13")
+    (pin "14")
+    (pin "15")
+    (pin "16")
+    (pin "2")
+    (pin "3")
+    (pin "4")
+    (pin "5")
+    (pin "6")
+    (pin "7")
+    (pin "8")
+    (pin "9")
   )
   (symbol (lib_id "power:GND") (at 45.72 124.46 0) (unit 1)
@@
     (pin "1")
   )
-  (symbol (lib_id "Device:LED_ALT") (at 46.99 48.26 180) (unit 1)
+  (symbol (lib_id "Device:LED") (at 46.99 48.26 180) (unit 1)
     (in_bom yes) (on_board yes)
     (property "Reference" "D34" (id 0) (at 46.99 50.8 0))
@@
       (effects (font (size 1.27 1.27)) hide)
     )
-    (property "Datasheet" "" (id 3) (at 46.99 48.26 0)
-      (effects (font (size 1.27 1.27)) hide)
-    )
-  )
-  (symbol (lib_id "Device:LED_ALT") (at 46.99 55.88 180) (unit 1)
+    (property "Datasheet" "~" (id 3) (at 46.99 48.26 0)
+      (effects (font (size 1.27 1.27)) hide)
+    )
+    (pin "1")
+    (pin "2")
+  )
+  (symbol (lib_id "Device:LED") (at 46.99 55.88 180) (unit 1)
     (in_bom yes) (on_board yes)
     (property "Reference" "D35" (id 0) (at 46.99 58.42 0))
@@
       (effects (font (size 1.27 1.27)) hide)
     )
-    (property "Datasheet" "" (id 3) (at 46.99 55.88 0)
-      (effects (font (size 1.27 1.27)) hide)
-    )
+    (property "Datasheet" "~" (id 3) (at 46.99 55.88 0)
+      (effects (font (size 1.27 1.27)) hide)
+    )
+    (pin "1")
+    (pin "2")
   )
   (symbol (lib_id "Device:R") (at 59.69 48.26 270) (unit 1)
@@
     (pin "2")
   )
-  (symbol (lib_id "Device:LED_ALT") (at 87.63 77.47 0) (unit 1)
+  (symbol (lib_id "Device:LED") (at 87.63 77.47 0) (unit 1)
     (in_bom yes) (on_board yes)
     (property "Reference" "D74" (id 0) (at 87.63 74.93 0))
@@
       (effects (font (size 1.27 1.27)) hide)
     )
-    (property "Datasheet" "" (id 3) (at 87.63 77.47 0)
-      (effects (font (size 1.27 1.27)) hide)
-    )
-  )
-  (symbol (lib_id "Device:LED_ALT") (at 87.63 82.55 0) (unit 1)
+    (property "Datasheet" "~" (id 3) (at 87.63 77.47 0)
+      (effects (font (size 1.27 1.27)) hide)
+    )
+    (pin "1")
+    (pin "2")
+  )
+  (symbol (lib_id "Device:LED") (at 87.63 82.55 0) (unit 1)
     (in_bom yes) (on_board yes)
     (property "Reference" "D75" (id 0) (at 87.63 80.01 0))
@@
       (effects (font (size 1.27 1.27)) hide)
     )
-    (property "Datasheet" "" (id 3) (at 87.63 82.55 0)
-      (effects (font (size 1.27 1.27)) hide)
-    )
-  )
-  (symbol (lib_id "Device:LED_ALT") (at 87.63 87.63 0) (unit 1)
+    (property "Datasheet" "~" (id 3) (at 87.63 82.55 0)
+      (effects (font (size 1.27 1.27)) hide)
+    )
+    (pin "1")
+    (pin "2")
+  )
+  (symbol (lib_id "Device:LED") (at 87.63 87.63 0) (unit 1)
     (in_bom yes) (on_board yes)
     (property "Reference" "D76" (id 0) (at 87.63 85.09 0))
@@
       (effects (font (size 1.27 1.27)) hide)
     )
-    (property "Datasheet" "" (id 3) (at 87.63 87.63 0)
-      (effects (font (size 1.27 1.27)) hide)
-    )
-  )
-  (symbol (lib_id "Device:LED_ALT") (at 87.63 92.71 0) (unit 1)
+    (property "Datasheet" "~" (id 3) (at 87.63 87.63 0)
+      (effects (font (size 1.27 1.27)) hide)
+    )
+    (pin "1")
+    (pin "2")
+  )
+  (symbol (lib_id "Device:LED") (at 87.63 92.71 0) (unit 1)
     (in_bom yes) (on_board yes)
     (property "Reference" "D77" (id 0) (at 87.63 90.17 0))
@@
       (effects (font (size 1.27 1.27)) hide)
     )
-    (property "Datasheet" "" (id 3) (at 87.63 92.71 0)
-      (effects (font (size 1.27 1.27)) hide)
-    )
-  )
-  (symbol (lib_id "Device:LED_ALT") (at 87.63 97.79 0) (unit 1)
+    (property "Datasheet" "~" (id 3) (at 87.63 92.71 0)
+      (effects (font (size 1.27 1.27)) hide)
+    )
+    (pin "1")
+    (pin "2")
+  )
+  (symbol (lib_id "Device:LED") (at 87.63 97.79 0) (unit 1)
     (in_bom yes) (on_board yes)
     (property "Reference" "D78" (id 0) (at 87.63 95.25 0))
@@
       (effects (font (size 1.27 1.27)) hide)
     )
-    (property "Datasheet" "" (id 3) (at 87.63 97.79 0)
-      (effects (font (size 1.27 1.27)) hide)
-    )
-  )
-  (symbol (lib_id "Device:LED_ALT") (at 87.63 102.87 0) (unit 1)
+    (property "Datasheet" "~" (id 3) (at 87.63 97.79 0)
+      (effects (font (size 1.27 1.27)) hide)
+    )
+    (pin "1")
+    (pin "2")
+  )
+  (symbol (lib_id "Device:LED") (at 87.63 102.87 0) (unit 1)
     (in_bom yes) (on_board yes)
     (property "Reference" "D79" (id 0) (at 87.63 100.33 0))
@@
       (effects (font (size 1.27 1.27)) hide)
     )
-    (property "Datasheet" "" (id 3) (at 87.63 102.87 0)
-      (effects (font (size 1.27 1.27)) hide)
-    )
-  )
-  (symbol (lib_id "Device:LED_ALT") (at 87.63 107.95 0) (unit 1)
+    (property "Datasheet" "~" (id 3) (at 87.63 102.87 0)
+      (effects (font (size 1.27 1.27)) hide)
+    )
+    (pin "1")
+    (pin "2")
+  )
+  (symbol (lib_id "Device:LED") (at 87.63 107.95 0) (unit 1)
     (in_bom yes) (on_board yes)
     (property "Reference" "D80" (id 0) (at 87.63 105.41 0))
@@
       (effects (font (size 1.27 1.27)) hide)
     )
-    (property "Datasheet" "" (id 3) (at 87.63 107.95 0)
-      (effects (font (size 1.27 1.27)) hide)
-    )
-  )
-  (symbol (lib_id "Device:LED_ALT") (at 87.63 113.03 0) (unit 1)
+    (property "Datasheet" "~" (id 3) (at 87.63 107.95 0)
+      (effects (font (size 1.27 1.27)) hide)
+    )
+    (pin "1")
+    (pin "2")
+  )
+  (symbol (lib_id "Device:LED") (at 87.63 113.03 0) (unit 1)
     (in_bom yes) (on_board yes)
     (property "Reference" "D81" (id 0) (at 87.63 110.49 0))
@@
       (effects (font (size 1.27 1.27)) hide)
     )
-    (property "Datasheet" "" (id 3) (at 87.63 113.03 0)
-      (effects (font (size 1.27 1.27)) hide)
-    )
+    (property "Datasheet" "~" (id 3) (at 87.63 113.03 0)
+      (effects (font (size 1.27 1.27)) hide)
+    )
+    (pin "1")
+    (pin "2")
   )
   (symbol (lib_id "Device:R") (at 77.47 77.47 270) (unit 1)

Commit message: Fix ALU
Parts:
- U16, U18: symbol 8bit-computer-rescue:74LS86 -> 74xx:74LS86
- U20, U21: symbol 8bit-computer-rescue:74LS283 -> 74xx:74LS283
- U22: symbol 8bit-computer-rescue:74LS02 -> 74xx:74LS02
Connections:
- net A_0: now also U21.5 (A1)
- net A_1: now also U21.3 (A2)
- net A_2: now also U21.14 (A3)
- net A_3: now also U21.12 (A4)
- net A_4: now also U20.5 (A1)
- net A_5: now also U20.3 (A2)
- net A_6: now also U20.14 (A3)
- net A_7: now also U20.12 (A4)
- net BUS_0: now also U17.11 (B7)
- net BUS_1: now also U17.12 (B6)
- net BUS_2: now also U17.13 (B5)
- net BUS_3: now also U17.14 (B4)
- net BUS_4: now also U17.15 (B3)
- net BUS_5: now also U17.16 (B2)
- net BUS_6: now also U17.17 (B1)
- net BUS_7: now also U17.18 (B0)
- net B_0: now also U18.12
- net B_1: now also U18.9
- net B_2: now also U18.4
- net B_3: now also U18.1
- net B_4: now also U16.12
- net B_5: now also U16.9
- net B_6: now also U16.4
- net B_7: now also U16.1
- net CF: now also U19.3 (Q0)
- net CLK: now also U19.7 (Cp)
- net CLR: now also U19.15 (Mr)
- net GND: now also U19.1 (Oe1), U19.2 (Oe2)
- net SU: now also U16.10, U16.13, U16.2, U16.5, U18.10, U18.13, U18.2, U18.5, U21.7 (C0)
- net VCC: now also U17.1 (A->B)
- net ZF: now also U19.4 (Q1)
- net ~{EO}: now also U17.19 (CE)
- net ~{FI}: now also U19.10 (E2), U19.9 (E1)
- net at U17.2 (A0): now also D74.2 (A), U20.10 (S4), U22.2
- net at U17.3 (A1): now also D75.2 (A), U20.13 (S3), U22.3
- net at U17.4 (A2): now also D76.2 (A), U20.1 (S2), U22.5
- net at U17.5 (A3): now also D77.2 (A), U20.4 (S1), U22.6
- net at U17.6 (A4): now also D78.2 (A), U21.10 (S4), U22.8
- net at U17.7 (A5): now also D79.2 (A), U21.13 (S3), U22.9
- net at U17.8 (A6): now also D80.2 (A), U21.1 (S2), U22.11
- net at U17.9 (A7): now also D81.2 (A), U21.4 (S1), U22.12
- net at U23.1: now also U22.1
- net at U23.2: now also U22.4
- net at U23.3: now also U23.4
- net at U23.5: now also U23.8
- net at U23.6: now also U19.13 (D1)
- net at U23.10: now also U22.13
- net at U23.9: now also U22.10
- net at U19.14 (D0): now also U20.9 (C4)
- new net: U16.3, U20.11 (B4)
- new net: U16.6, U20.15 (B3)
- new net: U16.8, U20.2 (B2)
- new net: U16.11, U20.6 (B1)
- new net: U20.7 (C0), U21.9 (C4)
- new net: U18.3, U21.11 (B4)
- new net: U18.6, U21.15 (B3)
- new net: U18.8, U21.2 (B2)
- new net: U18.11, U21.6 (B1)
Other:
- moved on the sheet: C14, C15, D34, D35, R48, R49, U19
