File: control.kicad_sch (KiCad schematic)
At the start: 59 parts

Commit message: Fix Clock
Parts:
- C22, C23: value (none) -> 0.1µF; footprint (none) -> Capacitor_THT:C_Disc_D4.3mm_W1.9mm_P5.00mm
- D50, D52, D53, D55, D56: value (none) -> GREEN; footprint (none) -> LED_THT:LED_D5.0mm
- D51, D54, D57: value (none) -> RED; footprint (none) -> LED_THT:LED_D5.0mm
- D58, D59, D60, D61, D62, D63, D64, D65, D66, D67, D68, D69, D70, D71, D72, D73: value (none) -> BLUE; footprint (none) -> LED_THT:LED_D5.0mm
- R67, R68, R69, R70, R71, R72, R73, R74, R76, R77, R78, R79, R80, R81, R82, R83, R84, R85, R86, R87, R88, R89, R90, R91: value (none) -> 220; footprint (none) -> Resistor_THT:R_Axial_DIN0207_L6.3mm_D2.5mm_P7.62mm_Horizontal
- R75: value (none) -> 1K; footprint (none) -> Resistor_THT:R_Axial_DIN0207_L6.3mm_D2.5mm_P7.62mm_Horizontal
- SW8: value (none) -> Reset; footprint (none) -> Button_Switch_THT:SW_PUSH_6mm_H5mm
- U47, U52: value (none) -> 28C16; footprint (none) -> Package_DIP:DIP-24_W15.24mm_Socket
- U48: value (none) -> 74LS161; footprint (none) -> Package_DIP:DIP-16_W7.62mm
- U49, U53: value (none) -> 74LS04; footprint (none) -> Package_DIP:DIP-14_W7.62mm; symbol 8bit-computer-rescue:74LS04 -> 74xx:74LS04
- U50: value (none) -> 74LS138; footprint (none) -> Package_DIP:DIP-16_W7.62mm
- U51: value (none) -> 74LS00; footprint (none) -> Package_DIP:DIP-14_W7.62mm

Commit message: Fix
Parts:
- D50, D51, D52, D53, D54, D55, D56, D57, D58, D59, D60, D61, D62, D63, D64, D65, D66, D67, D68, D69, D70, D71, D72, D73: symbol Device:LED_ALT -> Device:LED
- SW8: symbol 8bit-computer-rescue:SW_Push -> Switch:SW_Push
- U51: symbol 8bit-computer-rescue:74LS00 -> 74xx:74LS00
Connections:
- net CE: now also D70.2 (A)
- net HLT: now also D58.2 (A)
- net OI: now also D69.2 (A)
- net RI: now also D60.2 (A)
- net SU: now also D67.2 (A)
- net VCC: now also SW8.2
- net at R74.1: now also D57.1 (K)
- net at R75.1: now also SW8.1
- net at R76.1: now also D58.1 (K)
- net at R77.1: now also D59.1 (K)
- net at R78.1: now also D60.1 (K)
- net at R79.1: now also D61.1 (K)
- net at R80.1: now also D62.1 (K)
- net at R81.1: now also D63.1 (K)
- net at R82.1: now also D64.1 (K)
- net at R83.1: now also D65.1 (K)
- net at R84.1: now also D66.1 (K)
- net at R85.1: now also D67.1 (K)
- net at R86.1: now also D68.1 (K)
- net at R87.1: now also D69.1 (K)
- net at R88.1: now also D70.1 (K)
- net at R89.1: now also D71.1 (K)
- net at R90.1: now also D72.1 (K)
- net at R67.2: now also D50.2 (A)
- net at R70.2: now also D55.2 (A)
- net at R73.1: now also D54.1 (K)
- net at R91.1: now also D73.1 (K)
- net at R68.2: now also D52.2 (A)
- net at R69.2: now also D53.2 (A)
- net at R71.2: now also D56.2 (A)
- net at R72.1: now also D51.1 (K)

Commit message: Fix ALU
Parts:
- U48: symbol 8bit-computer-rescue:74LS161 -> 74xx:74LS161
- U50: symbol 8bit-computer-rescue:74LS138 -> 74xx:74LS138
Connections:
- net CLR: now also U51.11
- net GND: now also U50.4 (E1), U50.5 (E2)
- net VCC: now also U48.10 (CET), U48.7 (CEP), U48.9 (~{PE}), U50.6 (E3)
- net ~{AI}: now also U49.10
- net ~{AO}: now also U49.8
- net ~{BI}: now also U53.4
- net ~{CLK}: now also U48.2 (CP)
- net ~{CLR}: now also U51.12, U51.13, U51.4, U51.8
- net ~{CO}: now also U53.12
- net ~{EO}: now also U53.2
- net ~{FI}: now also U53.6
- net ~{II}: now also U49.12
- net ~{IO}: now also U49.6
- net ~{J}: now also U53.10
- net ~{MI}: now also U49.2
- net ~{RO}: now also U49.4
- net at D59.2 (A): now also U49.1
- net at D61.2 (A): now also U49.3
- net at D62.2 (A): now also U49.5
- net at D63.2 (A): now also U49.13
- net at D64.2 (A): now also U49.11
- net at D65.2 (A): now also U49.9
- net at D66.2 (A): now also U53.1
- net at D68.2 (A): now also U53.3
- net at D71.2 (A): now also U53.13
- net at D72.2 (A): now also U53.11
- net at D73.2 (A): now also U53.5
- net at U51.5: now also U50.10 (O5)
- net at U51.6: now also U51.1, U51.2
- net at U51.3: now also U48.1 (~{MR})
- net at U51.10: now also R75.1, SW8.1, U51.9
- net at D57.2 (A): now also U48.12 (Q2), U50.3 (A2)
- net at D54.2 (A): now also U48.13 (Q1), U50.2 (A1)
- net at D51.2 (A): now also U48.14 (Q0), U50.1 (A0)
- net at D50.1 (K): now also U50.11 (O4)
- net at D52.1 (K): now also U50.12 (O3)
- net at D53.1 (K): now also U50.13 (O2)
- net at D55.1 (K): now also U50.14 (O1)
- net at D56.1 (K): now also U50.15 (O0)
